File: CarteCaracASIC.kicad_pcb (KiCad board)
At the start: 4 copper layers, 150 x 250 mm, 148 parts, among them J1 Conn_02x25_Top_Bottom_Mountin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, U1 ASIC_JUICE

Commit message: Signaux ASIC sortis
Parts:
- moved CY1 16.3 mm to (20.8, 18.5)
- moved CY3 11.0 mm to (20.8, 14.4), turned to 180 degrees
- moved CY2 10.9 mm to (20.8, 10.3), turned to 180 degrees
- moved RX14 1.64 mm to (-5.37, 2.07)
- moved RthB0 1.27 mm to (3.18, 3.94)
- moved CX14 1.27 mm to (-1.06, 1.18)
- moved CX8 1.22 mm to (-7.14, 2.09), turned to 270 degrees
- moved RZ31 1.17 mm to (2.77, -1.70)
- moved CX13 0.62 mm to (-7.64, 6.12)
- moved RX33 0.58 mm to (-12.0, 26.5)
- moved RY33 0.58 mm to (-13.8, 26.5)
- moved RZ33 0.58 mm to (-10.2, 26.5)
- moved RX30 0.06 mm to (5.86, 9.98)
Routing:
- net /VDD_Y: track 1.93 -> 71.6 mm
- net /+6V_C: track 12.2 -> 76.5 mm
- net /+6V_B: track 13.2 -> 75.0 mm, vias 0 -> 2
- net /V_BIAS_LNA_Y: track 4.26 -> 64.5 mm, vias 0 -> 1
- net /Sy: track 1.74 -> 54.5 mm, vias 0 -> 1
- net /CR_Z: track 1.79 -> 53.3 mm, vias 0 -> 1
- net /V_BIAS_LNA_Z: track 3.92 -> 54.9 mm, vias 0 -> 1
- net /AsicFM/ChannelY/+32: track 0.00 -> 46.0 mm, vias 0 -> 1
- net /VDD_Z: track 14.8 -> 57.9 mm
- net /AsicFM/ChannelZ/+32: track 0.00 -> 40.3 mm, vias 0 -> 1
- net /M_Z: track 4.99 -> 43.8 mm
- net /AsicFM/Regu_Bias_LNA_Z: track 3.52 -> 40.2 mm, vias 0 -> 1
- net /CR_X: track 1.82 -> 38.2 mm, vias 0 -> 2
- net /B_Y: track 5.05 -> 41.4 mm
- net /RTNy: track 1.70 -> 37.4 mm, vias 0 -> 1
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- added copper zone on B.Cu, net GND
- added copper zone on F.Cu, net GND

Commit message: 20-12-19
Parts:
- SW_X32-34, SW_Y32-34, SW_Z32-34: footprint LibPersoNadj:Switch_4P3T_MRA403_NKK -> LibPersoNadj:Switch_4P3T_MRA403_NKK_Turned30°
- moved H7 372.9 mm to (169.4, 265.1), turned to 180 degrees
- moved CZ1 299.4 mm to (98.3, 262.5), turned to 180 degrees
- moved CY14 293.7 mm to (112.4, 254.0), turned to 0 degrees
- moved CZ3 291.6 mm to (98.3, 258.4), turned to 180 degrees
- moved H5 291.2 mm to (39.4, 265.1), turned to 180 degrees
- moved RY14 290.9 mm to (108.2, 254.3), turned to 270 degrees
- moved H8 289.5 mm to (169.4, 35.1), turned to 180 degrees
- moved RY41 286.6 mm to (105.2, 253.2), turned to 0 degrees
- moved CZ8 286.1 mm to (102.7, 253.9), turned to 270 degrees
- moved CY11 285.8 mm to (113.2, 249.3), turned to 0 degrees
- moved CY35 284.3 mm to (115.8, 247.2), turned to 0 degrees
- moved CZ2 283.9 mm to (98.3, 254.3), turned to 180 degrees
- moved CY10 283.7 mm to (109.8, 249.7), turned to 270 degrees
- moved CY_CR1 281.9 mm to (120.4, 243.4), turned to 270 degrees
- moved RY30 281.4 mm to (115.7, 245.6), turned to 180 degrees
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Routing:
- removed copper zone on F.Cu, net GND

Commit message: Del des point de tests et redimentionnement
Parts:
- removed TP_POT_BiasX1, TP_POT_BiasX2, TP_POT_BiasY1, TP_POT_BiasY2, TP_POT_BiasZ1, TP_POT_BiasZ2, TP_POT_VDDX1, TP_POT_VDDX2, TP_POT_VDDY1, TP_POT_VDDY2, TP_POT_VDDZ1, TP_POT_VDDZ2, TP_Pot_OffsetX1, TP_Pot_OffsetX2, TP_Pot_OffsetY1, TP_Pot_OffsetY2, TP_Pot_OffsetZ1, TP_Pot_OffsetZ2: TestPoint, Connector:Banana_Jack_1Pin
- moved H6 295.4 mm to (170.0, 300.0), turned to 0 degrees
- moved H8 294.8 mm to (40.0, 300.0), turned to 0 degrees
- moved J1 294.0 mm to (107.5, 312.0), turned to 0 degrees
- moved H5 273.3 mm to (170.0, 25.0), turned to 0 degrees
- moved H7 272.7 mm to (40.0, 25.0), turned to 0 degrees
- moved CZ1 235.2 mm to (111.1, 27.6), turned to 0 degrees
- moved CZ3 227.0 mm to (111.1, 31.7), turned to 0 degrees
- moved RVZ10 224.1 mm to (150.0, 270.0), turned to 0 degrees
- moved RVX10 223.6 mm to (60.0, 270.0), turned to 0 degrees
- moved CZ2 218.8 mm to (111.1, 35.8), turned to 0 degrees
- moved RY14 218.6 mm to (101.2, 35.8), turned to 90 degrees
- moved CY14 218.4 mm to (97.0, 36.1), turned to 180 degrees
- moved CZ8 217.7 mm to (106.7, 36.2), turned to 90 degrees
- moved RY41 216.3 mm to (104.2, 36.9), turned to 180 degrees
- moved CZ11 213.8 mm to (116.0, 38.8), turned to 90 degrees
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Connections:
- CX20 pad 2: /AsicFM/In2P_X -> /In2P_X
- CX_CR1 pad 2: /AsicFM/In2P_X -> /In2P_X
- CY20 pad 2: /AsicFM/In2P_Y -> /In2P_Y
- CY_CR1 pad 2: /AsicFM/In2P_Y -> /In2P_Y
- CZ20 pad 2: /AsicFM/In2P_Z -> /In2P_Z
- CZ_CR1 pad 2: /AsicFM/In2P_Z -> /In2P_Z
- J1 pad 17: Net-(J1-Pad17) -> /In2P_X
- J1 pad 18: Net-(J1-Pad18) -> /In2P_Y
- J1 pad 19: Net-(J1-Pad19) -> /In2P_Z
- RX20 pad 1: /AsicFM/In2P_X -> /In2P_X
- RY20 pad 1: /AsicFM/In2P_Y -> /In2P_Y
- RZ20 pad 1: /AsicFM/In2P_Z -> /In2P_Z
- SW_RX10 pad 1: Net-(SW_RX10-Pad1) -> /AsicFM/Pot_Bias_X_1
- SW_RX10 pad 4: Net-(SW_RX10-Pad4) -> /AsicFM/Pot_Bias_X_2
- SW_RX12 pad 1: Net-(SW_RX12-Pad1) -> /AsicFM/Pot_VDD_X_1
- SW_RX12 pad 4: Net-(SW_RX12-Pad4) -> /AsicFM/Pot_VDD_X_2
- SW_RY10 pad 1: Net-(SW_RY10-Pad1) -> /AsicFM/Pot_Bias_Y_1
- SW_RY10 pad 4: Net-(SW_RY10-Pad4) -> /AsicFM/Pot_Bias_Y_2
- SW_RY12 pad 1: Net-(SW_RY12-Pad1) -> /AsicFM/Pot_VDD_Y_1
- SW_RY12 pad 4: Net-(SW_RY12-Pad4) -> /AsicFM/Pot_VDD_Y_2
- SW_RZ10 pad 1: Net-(SW_RZ10-Pad1) -> /AsicFM/Pot_Bias_Z_1
- SW_RZ10 pad 4: Net-(SW_RZ10-Pad4) -> /AsicFM/Pot_Bias_Z_2
- SW_RZ12 pad 1: Net-(SW_RZ12-Pad1) -> /AsicFM/Pot_VDD_Z_1
- SW_RZ12 pad 4: Net-(SW_RZ12-Pad4) -> /AsicFM/Pot_VDD_Z_2
- SW_X32-34 pad 2: Net-(SW_X32-34-Pad2) -> /AsicFM/Pot_Offset_X_1
- SW_X32-34 pad 5: Net-(SW_X32-34-Pad5) -> /AsicFM/Pot_Offset_X_2
- SW_Y32-34 pad 2: Net-(SW_Y32-34-Pad2) -> /AsicFM/Pot_Offset_Y_1
- SW_Y32-34 pad 5: Net-(SW_Y32-34-Pad5) -> /AsicFM/Pot_Offset_Y_2
- SW_Z32-34 pad 2: Net-(SW_Z32-34-Pad2) -> /AsicFM/Pot_Offset_Z_1
- SW_Z32-34 pad 5: Net-(SW_Z32-34-Pad5) -> /AsicFM/Pot_Offset_Z_2
- U1 pad 26: /AsicFM/In2P_Z -> /In2P_Z
- U1 pad 29: /AsicFM/In2P_Z -> /In2P_Z
- U1 pad 4: /AsicFM/In2P_X -> /In2P_X
- U1 pad 51: /AsicFM/In2P_Y -> /In2P_Y
- U1 pad 53: /AsicFM/In2P_Y -> /In2P_Y
- U1 pad 7: /AsicFM/In2P_X -> /In2P_X
Routing:
- net /In2P_Z: track 0.00 -> 15.0 mm, vias 0 -> 1
- net /AsicFM/In2P_Z: track 15.0 -> 0.00 mm, vias 1 -> 0
- net /AsicFM/In2P_Y: track 11.6 -> 0.00 mm, vias 1 -> 0
- net /In2P_Y: track 0.00 -> 11.6 mm, vias 0 -> 1
- net /In2P_X: track 0.00 -> 9.35 mm
- net /AsicFM/In2P_X: track 9.35 -> 0.00 mm
- removed copper zone on B.Cu, net GND
Other:
- board size 150 x 250 mm -> 150 x 290 mm
