File: CarteCaracASIC_CQFP64/CarteCaracASIC.kicad_pcb (KiCad board)
At the start: 4 copper layers, 150 x 290 mm, 130 parts, among them J1 Conn_02x25_Top_Bottom_Mountin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, U1 ASIC_JUICE

Commit message: Added 2nd card
Parts:
- removed TP_6vX0, TP_6vY0, TP_6vZ0, TP_BZ0, TP_Cal0, TP_Mx0, TP_My0, TP_Mz0, TP_RTNx0, TP_RTNy0, TP_RTNz0, TP_Sx0, TP_Sy0, TP_Sz0, TP_VddX0, TP_VddY0, TP_VddZ0: TestPoint, Connector_PinHeader_2.54mm:PinHeader_1x01_P2.54mm_Vertical
- added SW_Channels_0: SW_6P3T_Slide6x3, LibPersoNadj:SW_6P3T_MSS6350R04_TE, F.Cu at (100.0, 365.0)
- added SW_Pot_0: SW_Slide_DP3T, LibPersoNadj:MHS233K_DP3T_Slide_Switch, F.Cu at (9.00, 267.5)
- TP_Pot1: renamed from TP_BX0; footprint Connector_PinHeader_2.54mm:PinHeader_1x01_P2.54mm_Vertical -> LibPersoNadj:Banana_test_point_4mm
- TP_Pot2: renamed from TP_BY0; footprint Connector_PinHeader_2.54mm:PinHeader_1x01_P2.54mm_Vertical -> LibPersoNadj:Banana_test_point_4mm
- moved TP_Pot2 227.8 mm to (50.0, 363.0), turned to 180 degrees
- moved TP_Pot1 211.6 mm to (70.0, 363.0), turned to 180 degrees
- moved J1 86.7 mm to (160.0, 381.0)
- moved H6 78.3 mm to (205.0, 370.0)
- moved H8 78.3 mm to (5.00, 370.0)
- moved RVX10 53.9 mm to (40.0, 320.0)
- moved RVX12 53.9 mm to (40.0, 267.5)
- moved RV_X32-34 53.9 mm to (40.0, 215.0)
- moved SW_RX10 53.9 mm to (40.0, 295.0)
- moved SW_RX12 53.9 mm to (40.0, 240.0)
- moved SW_X32-34 53.9 mm to (40.0, 180.0)
- moved RVZ10 51.0 mm to (160.0, 320.0)
- moved RVZ12 51.0 mm to (160.0, 267.5)
- moved RV_Z32-34 51.0 mm to (160.0, 215.0)
- moved SW_RZ10 51.0 mm to (160.0, 295.0)
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Connections:
- TP_Pot1 pad 1: /B_X -> /TP_Pot_1
- TP_Pot2 pad 1: /B_Y -> /TP_Pot_2
Other:
- board size 150 x 290 mm -> 210 x 360 mm

Commit message: Mise en forme de la carte + version carte ASIC et Carac separées
Parts:
- moved TP_Pot1 218.5 mm to (55.0, 145.0), turned to 270 degrees
- moved TP_Pot2 198.1 mm to (55.0, 165.0), turned to 270 degrees
- moved J1 191.9 mm to (0.00, 275.0)
- moved RV_Z32-34 187.4 mm to (25.0, 85.0), turned to 90 degrees
- moved SW_Z32-34 187.4 mm to (25.0, 50.0)
- moved H6 182.0 mm to (60.0, 260.0)
- moved SW_RZ12 180.6 mm to (25.0, 120.0)
- moved RVZ12 175.7 mm to (25.0, 155.0), turned to 90 degrees
- moved SW_Channels_0 171.6 mm to (53.0, 200.0), turned to 90 degrees
- moved SW_RZ10 171.0 mm to (25.0, 190.0)
- moved RV_Y32-34 170.3 mm to (-10.0, 85.0), turned to 90 degrees
- moved SW_Y32-34 170.3 mm to (-10.0, 50.0)
- moved RVZ10 165.1 mm to (25.0, 225.0), turned to 90 degrees
- moved SW_Pot_0 163.5 mm to (53.0, 110.0)
- moved SW_RY12 162.8 mm to (-10.0, 120.0)
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Other:
- board size 210 x 360 mm -> 130 x 300 mm
