File: CarteASIC_CQFP64/CarteASIC.sch (KiCad schematic (older format))
At the start: 6 parts, among them J1 Conn_02x34_Top_Bottom_Mountin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

Commit message: v0 near finished
Parts:
- removed J1: Conn_02x34_Top_Bottom_MountingPin, symbol Connector_Generic_MountingPin:Conn_02x34_Top_Bottom_MountingPin
- added J1: Conn_02x39_Top_Bottom_MountingPin, LibPersoNadj:db_78m_09565627813, symbol Connector_Generic_MountingPin:Conn_02x39_Top_Bottom_MountingPin
Connections:
- wire segments 156 -> 181
Other:
- note added: "Connecteur 78:\n\nFrom 15P(1-15):\nB*\nCR*\nPT1000 A\nM*\nSh*\n\n\nFrom 25S(26-50):\n\nRTN* (both)\nS*\nPT1000 A & B\nPWR_Shield*\n+6V*\nCAL\nCAL_RTN\nShield*\nCAL_Shield\n\n\nAdded:\n\nIn2P*\nV_Bias*\nVDD*\nR34* + & -\nR32* + & - ( - = +R34 )\nR12* + & - ( - = VDD )\nR10* + & - ( - = V_Bias )\n\n* for X Y and Z"
