File: CarteASIC_CQFP64/CarteASIC.kicad_pcb (KiCad board)
At the start: 4 copper layers, 130 x 300 mm, 115 parts, among them J1 Conn_02x25_Top_Bottom_Mountin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, U1 ASIC_JUICE

Commit message: v0 near finished
Parts:
- removed RVX10, RVY10, RVZ10: 12K, LibPersoNadj:Potentiometer_Bourns_3683S
- removed RVX12, RVY12, RVZ12: 16K, LibPersoNadj:Potentiometer_Bourns_3683S
- removed RV_X32-34, RV_Y32-34, RV_Z32-34: 5K, LibPersoNadj:Potentiometer_Bourns_3683S
- removed SW_Channels_0: SW_6P3T_Slide6x3, LibPersoNadj:SW_6P3T_MSS6350R04_TE
- removed SW_Pot_0: SW_Slide_DP3T, LibPersoNadj:MHS233K_DP3T_Slide_Switch
- removed SW_RX10, SW_RX12, SW_RY10, SW_RY12, SW_RZ10, SW_RZ12: SW_Push_DPDT, LibPersoNadj:SW_NKK_DPDT_B22AP
- removed SW_X32-34, SW_Y32-34, SW_Z32-34: SW_Rotary4x3, LibPersoNadj:Switch_4P3T_MRA403_NKK_Turned30°
- removed TP_Pot1, TP_Pot2: TestPoint, LibPersoNadj:Banana_test_point_4mm
- J1: value Conn_02x25_Top_Bottom_MountingPin -> Conn_02x39_Top_Bottom_MountingPin; footprint LibPersoNadj:DD50S564TLF -> LibPersoNadj:db_78m_09565627813
- moved J1 206.0 mm to (0.00, 69.0), turned to 180 degrees
- moved H6 191.0 mm to (40.0, 70.0)
- moved H8 191.0 mm to (-40.0, 70.0)
- moved H5 77.6 mm to (40.0, -30.0)
- moved H7 77.6 mm to (-40.0, -30.0)
Connections:
- CX10 pad 1: /V_BIAS_LNA_X -> /-RX10
- CX11 pad 1: /V_BIAS_LNA_X -> /-RX10
- CX12 pad 1: /VDD_X -> /-RX12
- CX13 pad 1: /VDD_X -> /-RX12
- CY10 pad 1: /V_BIAS_LNA_Y -> /-RY10
- CY11 pad 1: /V_BIAS_LNA_Y -> /-RY10
- CY12 pad 1: /VDD_Y -> /-RY12
- CY13 pad 1: /VDD_Y -> /-RY12
- CZ10 pad 1: /V_BIAS_LNA_Z -> /-RZ10
- CZ11 pad 1: /V_BIAS_LNA_Z -> /-RZ10
- CZ12 pad 1: /VDD_Z -> /-RZ12
- CZ13 pad 1: /VDD_Z -> /-RZ12
- J1 pad 16: Net-(J1-Pad16) -> /In2P_X
- J1 pad 17: /In2P_X -> /In2P_Y
- J1 pad 18: /In2P_Y -> /In2P_Z
- J1 pad 19: /In2P_Z -> /-RX10
- J1 pad 20: Net-(J1-Pad20) -> /-RY10
- J1 pad 21: Net-(J1-Pad21) -> /-RZ10
- J1 pad 22: Net-(J1-Pad22) -> /-RX12
- J1 pad 23: Net-(J1-Pad23) -> /-RY12
- J1 pad 24: Net-(J1-Pad24) -> /-RZ12
- J1 pad 25: Net-(J1-Pad25) -> GND
- RX10 pad 2: Net-(RX10-Pad2) -> /+RX10
- RX12 pad 2: Net-(RX12-Pad2) -> /+RX12
- RX31 pad 1: /AsicFM/ChannelX/+32 -> /+RX32
- RX31 pad 2: /VDD_X -> /-RX12
- RX33 pad 1: /AsicFM/ChannelX/-34 -> /-RX34
- RY10 pad 2: Net-(RY10-Pad2) -> /+RY10
- RY12 pad 2: Net-(RY12-Pad2) -> /+RY12
- RY31 pad 1: /AsicFM/ChannelY/+32 -> /+RY32
- RY31 pad 2: /VDD_Y -> /-RY12
- RY33 pad 1: /AsicFM/ChannelY/-34 -> /-RY34
- RZ10 pad 2: Net-(RZ10-Pad2) -> /+RZ10
- RZ12 pad 2: Net-(RZ12-Pad2) -> /+RZ12
- RZ31 pad 1: /AsicFM/ChannelZ/+32 -> /+RZ32
- RZ31 pad 2: /VDD_Z -> /-RZ12
- RZ33 pad 1: /AsicFM/ChannelZ/-34 -> /-RZ34
- U1 pad 11: /AsicFM/In2N_X -> /+RX34
- U1 pad 22: /AsicFM/In2N_Z -> /+RZ34
- U1 pad 33: /V_BIAS_LNA_Z -> /-RZ10
- U1 pad 34: /VDD_Z -> /-RZ12
- U1 pad 45: /VDD_Y -> /-RY12
- U1 pad 47: /V_BIAS_LNA_Y -> /-RY10
- U1 pad 56: /AsicFM/In2N_Y -> /+RY34
- U1 pad 63: /VDD_X -> /-RX12
- U1 pad 64: /V_BIAS_LNA_X -> /-RX10
Routing:
- net /-RY12: track 0.00 -> 159.3 mm, vias 0 -> 2
- net /+RY32: track 0.00 -> 154.8 mm, vias 0 -> 2
- net /-RY10: track 0.00 -> 147.1 mm, vias 0 -> 3
- net /-RZ10: track 0.00 -> 144.8 mm, vias 0 -> 3
- net /-RZ12: track 0.00 -> 141.5 mm, vias 0 -> 2
- net /+RX32: track 0.00 -> 120.3 mm, vias 0 -> 2
- net /-RZ34: track 0.00 -> 119.1 mm, vias 0 -> 1
- net /+RX10: track 0.00 -> 118.9 mm, vias 0 -> 2
- net /+RX12: track 0.00 -> 118.3 mm, vias 0 -> 2
- net /+RX34: track 0.00 -> 115.1 mm, vias 0 -> 2
- net /In2P_Y: track 11.6 -> 124.2 mm, vias 1 -> 3
- net /+RY12: track 0.00 -> 110.2 mm, vias 0 -> 1
- net /+RY10: track 0.00 -> 107.4 mm, vias 0 -> 1
- net /+RZ32: track 0.00 -> 103.9 mm, vias 0 -> 2
- net /+RY34: track 0.00 -> 102.9 mm, vias 0 -> 1
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- added copper zone on B.Cu, net GND
- added copper zone on F.Cu, net GND
- added copper zone on In1.Cu, net GND
- added copper zone on In2.Cu, net GND
Other:
- board size 130 x 300 mm -> 90 x 110 mm
- rule trace_min: 0.15 -> 0.2

Commit message: Mise en conformité valeurs PFM
Parts:
- CX10, CX12, CY10, CY12, CZ10, CZ12: value 150p -> 221p
- CX13, CY13, CZ13: value 220n/470n -> 470n
- CX20, CX_SC1, CX_SC2, CY20, CY_SC1, CY_SC2, CZ20, CZ_SC1, CZ_SC2: value TBD -> *
- CX35, CX36, CY35, CY36, CZ35, CZ36: value 1n -> *
- CX_CR1, CY_CR1, CZ_CR1: value TBD -> 150p
- RX14, RY14, RZ14: value 100 -> 400
- RX20, RY20, RZ20: value 68k -> 150k
- RX41, RY41, RZ41: value 49,9k -> 24,9k
Changed lines of the file:
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@@
       (effects (font (size 1 1) (thickness 0.15)) (justify mirror))
     )
-    (fp_text value 68k (at 0 -1.65 90) (layer B.Fab)
+    (fp_text value 150k (at 0 -1.65 90) (layer B.Fab)
       (effects (font (size 1 1) (thickness 0.15)) (justify mirror))
     )
@@
       (effects (font (size 1 1) (thickness 0.15)) (justify mirror))
     )
-    (fp_text value 68k (at 0 -1.65 90) (layer B.Fab)
+    (fp_text value 150k (at 0 -1.65 90) (layer B.Fab)
       (effects (font (size 1 1) (thickness 0.15)) (justify mirror))
     )
@@
       (effects (font (size 1 1) (thickness 0.15)) (justify mirror))
     )
-    (fp_text value 68k (at 0 -1.65) (layer B.Fab)
+    (fp_text value 150k (at 0 -1.65) (layer B.Fab)
       (effects (font (size 1 1) (thickness 0.15)) (justify mirror))
     )
@@
       (effects (font (size 1 1) (thickness 0.15)) (justify mirror))
     )
-    (fp_text value TBD (at 0 -1.43 90) (layer B.Fab)
+    (fp_text value * (at 0 -1.43 90) (layer B.Fab)
       (effects (font (size 1 1) (thickness 0.15)) (justify mirror))
     )
@@
       (effects (font (size 1 1) (thickness 0.15)) (justify mirror))
     )
-    (fp_text value TBD (at 0 -1.43 90) (layer B.Fab)
+    (fp_text value * (at 0 -1.43 90) (layer B.Fab)
       (effects (font (size 1 1) (thickness 0.15)) (justify mirror))
     )
@@
       (effects (font (size 1 1) (thickness 0.15)) (justify mirror))
     )
-    (fp_text value TBD (at 0 -1.43 90) (layer B.Fab)
+    (fp_text value 150p (at 0 -1.43 90) (layer B.Fab)
       (effects (font (size 1 1) (thickness 0.15)) (justify mirror))
     )
@@
       (effects (font (size 1 1) (thickness 0.15)) (justify mirror))
     )
-    (fp_text value 1n (at 0 -1.43 90) (layer B.Fab)
+    (fp_text value * (at 0 -1.43 90) (layer B.Fab)
       (effects (font (size 1 1) (thickness 0.15)) (justify mirror))
     )
@@
       (effects (font (size 1 1) (thickness 0.15)) (justify mirror))
     )
-    (fp_text value 1n (at 0 -1.43 90) (layer B.Fab)
+    (fp_text value * (at 0 -1.43 90) (layer B.Fab)
       (effects (font (size 1 1) (thickness 0.15)) (justify mirror))
     )
@@
       (effects (font (size 1 1) (thickness 0.15)) (justify mirror))
     )
-    (fp_text value TBD (at 0 -1.43 90) (layer B.Fab)
+    (fp_text value * (at 0 -1.43 90) (layer B.Fab)
       (effects (font (size 1 1) (thickness 0.15)) (justify mirror))
     )
@@
       (effects (font (size 1 1) (thickness 0.15)) (justify mirror))
     )
-    (fp_text value 220n/470n (at 0 -2.28) (layer B.Fab)
+    (fp_text value 470n (at 0 -2.28) (layer B.Fab)
       (effects (font (size 1 1) (thickness 0.15)) (justify mirror))
     )
@@
       (effects (font (size 1 1) (thickness 0.15)) (justify mirror))
     )
-    (fp_text value 150p (at 0 -1.43 90) (layer B.Fab)
+    (fp_text value 221p (at 0 -1.43 90) (layer B.Fab)
       (effects (font (size 1 1) (thickness 0.15)) (justify mirror))
     )
@@
       (effects (font (size 1 1) (thickness 0.15)) (justify mirror))
     )
-    (fp_text value 150p (at 0 -1.43 90) (layer B.Fab)
+    (fp_text value 221p (at 0 -1.43 90) (layer B.Fab)
       (effects (font (size 1 1) (thickness 0.15)) (justify mirror))
     )
@@
       (effects (font (size 1 1) (thickness 0.15)) (justify mirror))
     )
-    (fp_text value TBD (at 0 -1.43) (layer B.Fab)
+    (fp_text value * (at 0 -1.43) (layer B.Fab)
       (effects (font (size 1 1) (thickness 0.15)) (justify mirror))
     )
@@
       (effects (font (size 1 1) (thickness 0.15)) (justify mirror))
     )
-    (fp_text value TBD (at 0 -1.43) (layer B.Fab)
+    (fp_text value * (at 0 -1.43) (layer B.Fab)
       (effects (font (size 1 1) (thickness 0.15)) (justify mirror))
     )
@@
       (effects (font (size 1 1) (thickness 0.15)) (justify mirror))
     )
-    (fp_text value TBD (at 0 -1.43 90) (layer B.Fab)
+    (fp_text value 150p (at 0 -1.43 90) (layer B.Fab)
       (effects (font (size 1 1) (thickness 0.15)) (justify mirror))
     )
@@
       (effects (font (size 1 1) (thickness 0.15)) (justify mirror))
     )
-    (fp_text value 1n (at 0 -1.43 90) (layer B.Fab)
+    (fp_text value * (at 0 -1.43 90) (layer B.Fab)
       (effects (font (size 1 1) (thickness 0.15)) (justify mirror))
     )
@@
       (effects (font (size 1 1) (thickness 0.15)) (justify mirror))
     )
-    (fp_text value 1n (at 0 -1.43) (layer B.Fab)
+    (fp_text value * (at 0 -1.43) (layer B.Fab)
       (effects (font (size 1 1) (thickness 0.15)) (justify mirror))
     )
@@
       (effects (font (size 1 1) (thickness 0.15)) (justify mirror))
     )
-    (fp_text value TBD (at 0 -1.43 90) (layer B.Fab)
+    (fp_text value * (at 0 -1.43 90) (layer B.Fab)
       (effects (font (size 1 1) (thickness 0.15)) (justify mirror))
     )
@@
       (effects (font (size 1 1) (thickness 0.15)) (justify mirror))
     )
-    (fp_text value 220n/470n (at 0 -2.28 90) (layer B.Fab)
+    (fp_text value 470n (at 0 -2.28 90) (layer B.Fab)
       (effects (font (size 1 1) (thickness 0.15)) (justify mirror))
     )
@@
       (effects (font (size 1 1) (thickness 0.15)) (justify mirror))
     )
-    (fp_text value 150p (at 0 -1.43) (layer B.Fab)
+    (fp_text value 221p (at 0 -1.43) (layer B.Fab)
       (effects (font (size 1 1) (thickness 0.15)) (justify mirror))
     )
@@
       (effects (font (size 1 1) (thickness 0.15)) (justify mirror))
     )
-    (fp_text value 150p (at 0 -1.43 90) (layer B.Fab)
+    (fp_text value 221p (at 0 -1.43 90) (layer B.Fab)
       (effects (font (size 1 1) (thickness 0.15)) (justify mirror))
     )
@@
       (effects (font (size 1 1) (thickness 0.15)) (justify mirror))
     )
-    (fp_text value TBD (at 0 -1.43) (layer B.Fab)
+    (fp_text value * (at 0 -1.43) (layer B.Fab)
       (effects (font (size 1 1) (thickness 0.15)) (justify mirror))
     )
@@
       (effects (font (size 1 1) (thickness 0.15)) (justify mirror))
     )
-    (fp_text value TBD (at 0 -1.43) (layer B.Fab)
+    (fp_text value * (at 0 -1.43) (layer B.Fab)
       (effects (font (size 1 1) (thickness 0.15)) (justify mirror))
     )
@@
       (effects (font (size 1 1) (thickness 0.15)) (justify mirror))
     )
-    (fp_text value TBD (at 0 -1.43) (layer B.Fab)
+    (fp_text value 150p (at 0 -1.43) (layer B.Fab)
       (effects (font (size 1 1) (thickness 0.15)) (justify mirror))
     )
@@
       (effects (font (size 1 1) (thickness 0.15)) (justify mirror))
     )
-    (fp_text value 1n (at 0 -1.43 90) (layer B.Fab)
+    (fp_text value * (at 0 -1.43 90) (layer B.Fab)
       (effects (font (size 1 1) (thickness 0.15)) (justify mirror))
     )
@@
       (effects (font (size 1 1) (thickness 0.15)) (justify mirror))
     )
-    (fp_text value 1n (at 0 -1.43) (layer B.Fab)
+    (fp_text value * (at 0 -1.43) (layer B.Fab)
       (effects (font (size 1 1) (thickness 0.15)) (justify mirror))
     )
@@
       (effects (font (size 1 1) (thickness 0.15)) (justify mirror))
     )
-    (fp_text value TBD (at 0 -1.43) (layer B.Fab)
+    (fp_text value * (at 0 -1.43) (layer B.Fab)
       (effects (font (size 1 1) (thickness 0.15)) (justify mirror))
     )
@@
       (effects (font (size 1 1) (thickness 0.15)) (justify mirror))
     )
-    (fp_text value 220n/470n (at 0 -2.28) (layer B.Fab)
+    (fp_text value 470n (at 0 -2.28) (layer B.Fab)
       (effects (font (size 1 1) (thickness 0.15)) (justify mirror))
     )
@@
       (effects (font (size 1 1) (thickness 0.15)) (justify mirror))
     )
-    (fp_text value 150p (at 0 -1.43) (layer B.Fab)
+    (fp_text value 221p (at 0 -1.43) (layer B.Fab)
       (effects (font (size 1 1) (thickness 0.15)) (justify mirror))
     )
@@
       (effects (font (size 1 1) (thickness 0.15)) (justify mirror))
     )
-    (fp_text value 150p (at 0 -1.43 90) (layer B.Fab)
+    (fp_text value 221p (at 0 -1.43 90) (layer B.Fab)
       (effects (font (size 1 1) (thickness 0.15)) (justify mirror))
     )
@@
       (effects (font (size 0.6 0.6) (thickness 0.15)) (justify mirror))
     )
-    (fp_text value 49,9k (at 0 -1.43 90) (layer B.Fab)
+    (fp_text value 24,9k (at 0 -1.43 90) (layer B.Fab)
       (effects (font (size 1 1) (thickness 0.15)) (justify mirror))
     )
@@
       (effects (font (size 0.6 0.6) (thickness 0.15)) (justify mirror))
     )
-    (fp_text value 100 (at 0 -1.43) (layer B.Fab)
+    (fp_text value 400 (at 0 -1.43) (layer B.Fab)
       (effects (font (size 1 1) (thickness 0.15)) (justify mirror))
     )
@@
       (effects (font (size 0.6 0.6) (thickness 0.15)) (justify mirror))
     )
-    (fp_text value 49,9k (at 0 -1.43) (layer B.Fab)
+    (fp_text value 24,9k (at 0 -1.43) (layer B.Fab)
       (effects (font (size 1 1) (thickness 0.15)) (justify mirror))
     )
@@
       (effects (font (size 0.6 0.6) (thickness 0.15)) (justify mirror))
     )
-    (fp_text value 100 (at 0 -1.43 90) (layer B.Fab)
+    (fp_text value 400 (at 0 -1.43 90) (layer B.Fab)
       (effects (font (size 1 1) (thickness 0.15)) (justify mirror))
     )
@@
       (effects (font (size 0.6 0.6) (thickness 0.15)) (justify mirror))
     )
-    (fp_text value 49,9k (at 0 -1.43) (layer B.Fab)
+    (fp_text value 24,9k (at 0 -1.43) (layer B.Fab)
       (effects (font (size 1 1) (thickness 0.15)) (justify mirror))
     )
@@
       (effects (font (size 0.6 0.6) (thickness 0.15)) (justify mirror))
     )
-    (fp_text value 100 (at 0 -1.43 90) (layer B.Fab)
-      (effects (font (size 1 1) (thickness 0.15)) (justify mirror))
-    )
+    (fp_text value 400 (at 0 -1.43 90) (layer B.Fab)
+      (effects (font (size 1 1) (thickness 0.15)) (justify mirror))
+    )
