File: CarteCaracTo/CarteCaracTo.kicad_pcb (KiCad board)
At the start: 6 copper layers, 130 x 125.1 mm, 213 parts, among them J1 Conn_02x10_Counter_Clockwise, J11 Conn_02x10_Counter_Clockwise, J21 Conn_02x05_Counter_Clockwise, J26 Conn_02x05_Counter_Clockwise, J31 Conn_02x10_Counter_Clockwise, J41 Conn_02x10_Counter_Clockwise, J50 Sub-D50_F, J51 DB15_Male_MountingHoles, J52 DB25_Female_MountingHoles

Commit message: mineur
Parts:
- added J2: Conn_01x01, Connector_Coaxial:BNC_Amphenol_B6252HB-NPP3G-50_Horizontal, F.Cu at (186.0, -1.00)
- added J3: Conn_Coaxial, Connector_Coaxial:BNC_Amphenol_B6252HB-NPP3G-50_Horizontal, F.Cu at (169.2, -1.00)
- added J4: Conn_Coaxial, Connector_Coaxial:BNC_Amphenol_B6252HB-NPP3G-50_Horizontal, F.Cu at (152.5, -1.00)
- added J5: Conn_Coaxial, Connector_Coaxial:BNC_Amphenol_B6252HB-NPP3G-50_Horizontal, F.Cu at (135.8, -1.00)
- added J6: Conn_Coaxial, Connector_Coaxial:BNC_Amphenol_B6252HB-NPP3G-50_Horizontal, F.Cu at (119.0, -1.00)
- added J7: Conn_Coaxial, Connector_Coaxial:BNC_Amphenol_B6252HB-NPP3G-50_Horizontal, F.Cu at (102.2, -1.00)
- added J8: Conn_Coaxial, Connector_Coaxial:BNC_Amphenol_B6252HB-NPP3G-50_Horizontal, F.Cu at (85.5, -1.00)
- added JGSE0: DB25_Male_MountingHoles, LibPersoNadj:DCCM25PCBRPN, F.Cu at (129.6, 13.8)
- added JMatrice0: DB25_Male_MountingHoles, LibPersoNadj:DCCM25PCBRPN, F.Cu at (94.6, 13.8)
- added R1: R, Resistor_SMD:R_0603_1608Metric_Pad1.05x0.95mm_HandSolder, F.Cu at (88.4, 43.6)
- added R10: R, Resistor_SMD:R_0603_1608Metric_Pad1.05x0.95mm_HandSolder, F.Cu at (113.8, 38.6)
- added R11: R, Resistor_SMD:R_0603_1608Metric_Pad1.05x0.95mm_HandSolder, F.Cu at (109.5, 38.6)
- added R12: R, Resistor_SMD:R_0603_1608Metric_Pad1.05x0.95mm_HandSolder, F.Cu at (109.5, 41.1)
- added R2: R, Resistor_SMD:R_0603_1608Metric_Pad1.05x0.95mm_HandSolder, F.Cu at (88.4, 38.6)
- added R3: R, Resistor_SMD:R_0603_1608Metric_Pad1.05x0.95mm_HandSolder, F.Cu at (92.7, 38.6)
- added R4: R, Resistor_SMD:R_0603_1608Metric_Pad1.05x0.95mm_HandSolder, F.Cu at (88.4, 41.1)
- added R5: R, Resistor_SMD:R_0603_1608Metric_Pad1.05x0.95mm_HandSolder, F.Cu at (215.3, -29.1)
- added R6: R, Resistor_SMD:R_0603_1608Metric_Pad1.05x0.95mm_HandSolder, F.Cu at (219.7, -34.1)
- added R7: R, Resistor_SMD:R_0603_1608Metric_Pad1.05x0.95mm_HandSolder, F.Cu at (215.3, -31.6)
- added R8: R, Resistor_SMD:R_0603_1608Metric_Pad1.05x0.95mm_HandSolder, F.Cu at (215.3, -34.1)
- added R9: R, Resistor_SMD:R_0603_1608Metric_Pad1.05x0.95mm_HandSolder, F.Cu at (109.5, 43.6)
- added SW1: SW_3PDT, LibPersoNadj:SW_3PDT_M2032TNW01_NKK, F.Cu at (156.6, 17.8)
- added SW2: SW_DIP_x05, Button_Switch_THT:SW_DIP_SPSTx05_Slide_9.78x14.88mm_W7.62mm_P2.54mm, F.Cu at (188.4, 5.45)
- added SW3: SW_Slide_DP3T, LibPersoNadj:Switch_DP3T_Slide_MHS233K, F.Cu at (171.2, 11.5)
- added SW4: SW_SPDT, LibPersoNadj:SW_SPDT_B12AP_NKK, F.Cu at (81.3, 25.0)
- added SW5: SW_SPDT, LibPersoNadj:SW_SPDT_B12AP_NKK, F.Cu at (89.6, 25.0)
- added SW6: SW_SPDT, LibPersoNadj:SW_SPDT_B12AP_NKK, F.Cu at (97.9, 25.0)
- added SW7: SW_3PDT, LibPersoNadj:Switch_DP3T_Slide_MHS233K, F.Cu at (181.4, 11.5)
- added SW_RegB0: SW_Push_DPDT, LibPersoNadj:SW_DPDT_B22AP_NKK, F.Cu at (208.6, -30.8)
- added SW_Rej_A0: SW_Push_DPDT, LibPersoNadj:SW_DPDT_B22AP_NKK, F.Cu at (81.7, 41.9)
- added SW_Rej_C0: SW_Push_DPDT, LibPersoNadj:SW_DPDT_B22AP_NKK, F.Cu at (102.8, 41.9)
- added U1: OPA4376, Package_SO:SOIC-14_3.9x8.7mm_P1.27mm, F.Cu at (106.3, 24.9)
Connections:
- J26 pad 4: /29 -> /27
- J31 pad 4: /34 -> /+6V_B
- J41 pad 5: /45 -> /+6V_A
- J41 pad 8: /48 -> /+6V_C
- J50 pad 0: Net-(J50-Pad0) -> GND
- J50 pad 29: /29 -> /27
- J50 pad 34: /34 -> /+6V_B
- J50 pad 45: /45 -> /+6V_A
- J50 pad 48: /48 -> /+6V_C
- J51 pad 0: Net-(J51-Pad0) -> GND
- J51 pad 1: /1 -> /101
- J51 pad 10: /10 -> /110
- J51 pad 11: /11 -> /111
- J51 pad 12: /12 -> /112
- J51 pad 13: /13 -> /113
- J51 pad 14: /14 -> /114
- J51 pad 15: /15 -> /115
- J51 pad 2: /2 -> /102
- J51 pad 3: /3 -> /103
- J51 pad 4: /4 -> /104
- J51 pad 5: /5 -> /105
- J51 pad 6: /6 -> /106
- J51 pad 7: /7 -> /107
- J51 pad 8: /8 -> /108
- J51 pad 9: /9 -> /109
- J52 pad 0: Net-(J52-Pad0) -> GND
- J52 pad 1: /26 -> /126
- J52 pad 10: /35 -> /135
- J52 pad 11: /36 -> /136
- J52 pad 12: /37 -> /137
- J52 pad 13: /38 -> /138
- J52 pad 14: /39 -> /139
- J52 pad 15: /40 -> /140
- J52 pad 16: /41 -> /141
- J52 pad 17: /42 -> /142
- J52 pad 18: /43 -> /143
- J52 pad 19: /44 -> /144
- J52 pad 2: /27 -> /127
- J52 pad 20: /45 -> /145
- J52 pad 21: /46 -> /146
- J52 pad 22: /47 -> /147
- J52 pad 23: /48 -> /148
- J52 pad 24: /49 -> /149
- J52 pad 25: /50 -> /150
- J52 pad 3: /28 -> /128
- J52 pad 4: /29 -> /129
- J52 pad 5: /30 -> /130
- J52 pad 6: /31 -> /131
- J52 pad 7: /32 -> /132
- J52 pad 8: /33 -> /133
- J52 pad 9: /34 -> /134
- TP107 pad 1: /29 -> /27
- TP108 pad 1: /29 -> /27
- TP147 pad 1: /34 -> /+6V_B
- TP148 pad 1: /34 -> /+6V_B
- TP189 pad 1: /45 -> /+6V_A
- TP190 pad 1: /45 -> /+6V_A
- TP195 pad 1: /48 -> /+6V_C
- TP196 pad 1: /48 -> /+6V_C

Commit message: Mise en forme de la carte + version carte ASIC et Carac separées
Parts:
- added J12v0: Conn_Coaxial, Connector_Coaxial:SMB_Jack_Vertical, F.Cu at (127.0, 40.0)
- JGSE0, JMatrice0: footprint LibPersoNadj:DCCM25PCBRPN -> Connector_Dsub:DSUB-25_Male_Horizontal_P2.77x2.84mm_EdgePinOffset9.90mm_Housed_MountingHolesOffset11.32mm
- SW7: footprint LibPersoNadj:Switch_DP3T_Slide_MHS233K -> LibPersoNadj:SW_3PDT_M2032TNW01_NKK
- moved TP222 328.2 mm to (241.8, 163.5), turned to 0 degrees
- moved TP221 325.5 mm to (236.8, 163.5), turned to 0 degrees
- moved TP224 321.6 mm to (241.8, 158.4), turned to 0 degrees
- moved TP223 318.9 mm to (236.8, 158.4), turned to 0 degrees
- moved TP242 316.3 mm to (216.4, 163.5), turned to 0 degrees
- moved TP226 315.0 mm to (241.8, 153.3), turned to 0 degrees
- moved TP241 314.4 mm to (211.3, 163.5), turned to 0 degrees
- moved TP225 312.2 mm to (236.8, 153.3), turned to 0 degrees
- moved TP102 310.2 mm to (198.7, 163.5), turned to 0 degrees
- moved TP244 309.4 mm to (216.4, 158.4), turned to 0 degrees
- moved TP101 308.8 mm to (193.6, 163.5), turned to 0 degrees
- moved TP228 308.4 mm to (241.8, 148.2), turned to 0 degrees
- moved TP243 307.4 mm to (211.3, 158.4), turned to 0 degrees
- moved TP227 305.5 mm to (236.8, 148.2), turned to 0 degrees
- moved TP112 304.9 mm to (173.2, 163.5), turned to 0 degrees
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Connections:
- JGSE0 pad 22: /+12v -> Net-(JGSE0-Pad22)
- SW_Rej_C0 pad 5: /Source+6V_B -> /Source+6V_C
Other:
- board size 130 x 125.1 mm -> 262.5 x 167.5 mm
- board text added: "12V"
- board text added: "Analyseur 1"
- board text added: "Analyseur 2"
- board text added: "Analyseur 3"
- board text added: "Fonction transfer In"
- board text added: "Fonction transfer Out"
- board text added: "Manuel"
- board text added: "Matrice"
- board text added: "Normal"
- board text added: "Réjection"
- board text added: "S X Y RTN Z"
- board text added: "Sy RTNy"
- board text added: "Sz RTNz"
- board text added: "Test réjection"
- board text added: "X"
- board text added: "X Y Z"
- board text added: "X Y Z Y Z"
- board text added: "Y"
- board text added: "Z"
- board text added: "{"

Commit message: ID des pins, option capa sur sortie, option GND ou plan de masse sur BNC
Parts:
- removed J2: Conn_01x01, Connector_Coaxial:BNC_Amphenol_B6252HB-NPP3G-50_Horizontal
- added C1: C, Capacitor_SMD:C_0805_2012Metric_Pad1.15x1.40mm_HandSolder, F.Cu at (24.0, 87.0)
- added C2: C, Capacitor_SMD:C_0805_2012Metric_Pad1.15x1.40mm_HandSolder, F.Cu at (24.0, 62.0)
- added C3: C, Capacitor_SMD:C_0805_2012Metric_Pad1.15x1.40mm_HandSolder, F.Cu at (24.0, 37.0)
- added JDec_SA1: Conn_01x03, Connector_PinHeader_2.54mm:PinHeader_1x03_P2.54mm_Vertical, F.Cu at (30.0, 87.5)
- added JDec_SA2: Conn_01x03, Connector_PinHeader_2.54mm:PinHeader_1x03_P2.54mm_Vertical, F.Cu at (30.0, 62.5)
- added JDec_SA3: Conn_01x03, Connector_PinHeader_2.54mm:PinHeader_1x03_P2.54mm_Vertical, F.Cu at (30.0, 37.5)
- added JGND_I_SA1: Conn_01x03, Connector_PinHeader_2.54mm:PinHeader_1x03_P2.54mm_Vertical, F.Cu at (15.0, 50.0)
- added JGND_I_SA2: Conn_01x03, Connector_PinHeader_2.54mm:PinHeader_1x03_P2.54mm_Vertical, F.Cu at (15.0, 75.0)
- added JGND_I_SA3: Conn_01x03, Connector_PinHeader_2.54mm:PinHeader_1x03_P2.54mm_Vertical, F.Cu at (15.0, 100.0)
- added JGND_O_SA1: Conn_01x03, Connector_PinHeader_2.54mm:PinHeader_1x03_P2.54mm_Vertical, F.Cu at (15.0, 125.0)
- added JGND_O_SA2: Conn_01x03, Connector_PinHeader_2.54mm:PinHeader_1x03_P2.54mm_Vertical, F.Cu at (15.0, 150.0)
- added JGND_O_SA3: Conn_01x03, Connector_PinHeader_2.54mm:PinHeader_1x03_P2.54mm_Vertical, F.Cu at (15.0, 175.0)
- added JMasse0: Conn_01x02, Connector_PinHeader_2.54mm:PinHeader_1x02_P2.54mm_Vertical, F.Cu at (134.5, 110.5)
- added J_12v0: Conn_01x01, Connector_PinHeader_2.54mm:PinHeader_1x01_P2.54mm_Vertical, F.Cu at (136.0, 37.5)
- added J_I_SA1: Conn_01x01, Connector_PinHeader_2.54mm:PinHeader_1x01_P2.54mm_Vertical, F.Cu at (15.0, 40.0)
- added J_I_SA2: Conn_01x01, Connector_PinHeader_2.54mm:PinHeader_1x01_P2.54mm_Vertical, F.Cu at (15.0, 65.0)
- added J_I_SA3: Conn_01x01, Connector_PinHeader_2.54mm:PinHeader_1x01_P2.54mm_Vertical, F.Cu at (15.0, 90.0)
- added J_O_SA1: Conn_01x01, Connector_PinHeader_2.54mm:PinHeader_1x01_P2.54mm_Vertical, F.Cu at (15.0, 115.0)
- added J_O_SA2: Conn_01x01, Connector_PinHeader_2.54mm:PinHeader_1x01_P2.54mm_Vertical, F.Cu at (15.0, 141.0)
- added J_O_SA3: Conn_01x01, Connector_PinHeader_2.54mm:PinHeader_1x01_P2.54mm_Vertical, F.Cu at (15.0, 165.0)
- added J_Perturb0: Conn_Coaxial, Connector_Coaxial:BNC_Amphenol_B6252HB-NPP3G-50_Horizontal, F.Cu at (150.0, 30.0)
- added J_Perturb1: Conn_01x01, Connector_PinHeader_2.54mm:PinHeader_1x01_P2.54mm_Vertical, F.Cu at (150.0, 37.5)
- moved SW_Rej_C0 30.9 mm to (150.0, 65.0)
- moved SW_Rej_A0 29.0 mm to (122.0, 65.0)
- moved SW3 15.0 mm to (62.0, 40.0)
- moved SW4 15.0 mm to (39.5, 40.0)
- moved SW5 15.0 mm to (39.5, 65.0)
- moved SW6 15.0 mm to (39.5, 89.0)
- moved J12v0 11.7 mm to (136.0, 47.5)
- moved SW_RegB0 7.57 mm to (136.0, 65.0)
- moved R1 7.50 mm to (155.0, 41.9)
- moved R10 7.50 mm to (145.9, 53.7)
- moved R11 7.50 mm to (149.3, 53.7)
- moved R12 7.50 mm to (144.9, 50.0)
- moved R2 7.50 mm to (153.3, 41.9)
- moved R3 7.50 mm to (151.7, 41.9)
- moved R4 7.50 mm to (156.1, 46.4)
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Connections:
- J1 pad 10: /10 -> GND
- J1 pad 11: /110 -> GND
- J1 pad 7: /7 -> /43
- J1 pad 8: /8 -> /31
- J11 pad 16: /115 -> GND
- J11 pad 17: /114 -> GND
- J11 pad 19: /112 -> GND
- J11 pad 2: /12 -> GND
- J11 pad 4: /14 -> GND
- J11 pad 5: /15 -> GND
- J26 pad 3: /28 -> GND
- J26 pad 4: /27 -> /29
- J26 pad 8: /128 -> GND
- J3 pad 1: /Spectro1_In -> Net-(C3-Pad1)
- J3 pad 2: GND -> Net-(J3-Pad2)
- J31 pad 12: /139 -> GND
- J31 pad 13: /138 -> GND
- J31 pad 15: /136 -> GND
- J31 pad 16: /135 -> GND
- J31 pad 18: /133 -> GND
- J31 pad 3: /33 -> GND
- J31 pad 5: /35 -> GND
- J31 pad 6: /36 -> GND
- J31 pad 8: /38 -> GND
- J31 pad 9: /39 -> GND
- J4 pad 1: /Spectro2_In -> Net-(C2-Pad1)
- J4 pad 2: GND -> Net-(J4-Pad2)
- J41 pad 10: /50 -> GND
- J41 pad 11: /150 -> GND
- J41 pad 12: /149 -> GND
- J41 pad 14: /147 -> GND
- J41 pad 15: /146 -> GND
- J41 pad 19: /142 -> GND
- J41 pad 2: /42 -> GND
- J41 pad 6: /46 -> GND
- J41 pad 7: /47 -> GND
- J41 pad 9: /49 -> GND
- J5 pad 1: /Spectro3_In -> Net-(C1-Pad1)
- J5 pad 2: GND -> Net-(J5-Pad2)
- J50 pad 10: /10 -> GND
- J50 pad 12: /12 -> GND
- J50 pad 14: /14 -> GND
- J50 pad 15: /15 -> GND
- J50 pad 28: /28 -> GND
- J50 pad 29: /27 -> /29
- J50 pad 33: /33 -> GND
- J50 pad 35: /35 -> GND
- J50 pad 36: /36 -> GND
- J50 pad 38: /38 -> GND
- J50 pad 39: /39 -> GND
- J50 pad 42: /42 -> GND
- J50 pad 46: /46 -> GND
- J50 pad 47: /47 -> GND
- J50 pad 49: /49 -> GND
- J50 pad 50: /50 -> GND
- J50 pad 7: /7 -> /43
- J50 pad 8: /8 -> /31
- J51 pad 10: /110 -> GND
- J51 pad 12: /112 -> GND
- J51 pad 14: /114 -> GND
- J51 pad 15: /115 -> GND
- J52 pad 10: /135 -> GND
- J52 pad 11: /136 -> GND
- J52 pad 13: /138 -> GND
- J52 pad 14: /139 -> GND
- J52 pad 17: /142 -> GND
- J52 pad 21: /146 -> GND
- J52 pad 22: /147 -> GND
- J52 pad 24: /149 -> GND
- J52 pad 25: /150 -> GND
- J52 pad 3: /128 -> GND
- J52 pad 8: /133 -> GND
- JGSE0 pad 1: Net-(JGSE0-Pad1) -> /27
- JGSE0 pad 10: Net-(JGSE0-Pad10) -> /19
- JGSE0 pad 11: Net-(JGSE0-Pad11) -> /20
- JGSE0 pad 12: Net-(JGSE0-Pad12) -> /21
- JGSE0 pad 13: Net-(JGSE0-Pad13) -> GND
- JGSE0 pad 14: Net-(JGSE0-Pad14) -> /22
- JGSE0 pad 15: Net-(JGSE0-Pad15) -> /23
- JGSE0 pad 16: Net-(JGSE0-Pad16) -> /24
- JGSE0 pad 2: Net-(JGSE0-Pad2) -> /26
- JGSE0 pad 20: Net-(JGSE0-Pad20) -> GND
- JGSE0 pad 21: Net-(JGSE0-Pad21) -> GND
- JGSE0 pad 22: Net-(JGSE0-Pad22) -> GND
- JGSE0 pad 23: Net-(JGSE0-Pad23) -> GND
- JGSE0 pad 24: Net-(JGSE0-Pad24) -> GND
- JGSE0 pad 25: Net-(JGSE0-Pad25) -> GND
- JGSE0 pad 3: Net-(JGSE0-Pad3) -> /9
- JGSE0 pad 4: Net-(JGSE0-Pad4) -> /40
- JGSE0 pad 5: Net-(JGSE0-Pad5) -> /41
- JGSE0 pad 6: Net-(JGSE0-Pad6) -> /11
- JGSE0 pad 7: Net-(JGSE0-Pad7) -> /29
- JGSE0 pad 8: Net-(JGSE0-Pad8) -> /30
- JGSE0 pad 9: Net-(JGSE0-Pad9) -> /13
- JMatrice0 pad 1: /SpectroToMatrice -> /1
- JMatrice0 pad 10: /MatriceToSpectro3 -> /41
- JMatrice0 pad 12: Net-(JMatrice0-Pad12) -> /30
- JMatrice0 pad 17: Net-(JMatrice0-Pad17) -> /Spectro1ToMatrice
- JMatrice0 pad 18: Net-(JMatrice0-Pad18) -> /MatriceToSpectro1
- JMatrice0 pad 19: Net-(JMatrice0-Pad19) -> /Spectro2ToMatrice
- JMatrice0 pad 2: /1 -> /27
- JMatrice0 pad 20: Net-(JMatrice0-Pad20) -> /MatriceToSpectro2
- JMatrice0 pad 21: Net-(JMatrice0-Pad21) -> /Spectro3ToMatrice
- JMatrice0 pad 22: Net-(JMatrice0-Pad22) -> /MatriceToSpectro3
- JMatrice0 pad 4: /5 -> /40
- JMatrice0 pad 5: /Spectro1ToMatrice -> /5
- JMatrice0 pad 6: /Spectro2ToMatrice -> /29
- JMatrice0 pad 7: /Spectro3ToMatrice -> Net-(JMatrice0-Pad7)
- JMatrice0 pad 8: /MatriceToSpectro1 -> /26
- JMatrice0 pad 9: /MatriceToSpectro2 -> Net-(JMatrice0-Pad9)
- SW3 pad 0: Net-(SW3-Pad0) -> GND
- SW3 pad 1: /Sx -> /27
- SW3 pad 4: /27 -> /29
- SW6 pad 1: /27 -> /29
- SW_Rej_C0 pad 2: /+6V_B -> /+6V_C
- TP105 pad 1: /28 -> GND
- TP106 pad 1: /28 -> GND
- TP107 pad 1: /27 -> /29
- TP108 pad 1: /27 -> /29
- TP115 pad 1: /128 -> GND
- TP116 pad 1: /128 -> GND
- TP145 pad 1: /33 -> GND
- TP146 pad 1: /33 -> GND
- TP149 pad 1: /35 -> GND
- TP150 pad 1: /35 -> GND
- TP151 pad 1: /36 -> GND
- TP152 pad 1: /36 -> GND
- TP155 pad 1: /38 -> GND
- TP156 pad 1: /38 -> GND
- TP165 pad 1: /133 -> GND
- TP166 pad 1: /133 -> GND
- TP169 pad 1: /135 -> GND
- TP170 pad 1: /135 -> GND
- TP171 pad 1: /136 -> GND
- TP172 pad 1: /136 -> GND
- TP175 pad 1: /138 -> GND
- TP176 pad 1: /138 -> GND
- TP183 pad 1: /42 -> GND
- TP184 pad 1: /42 -> GND
- TP191 pad 1: /46 -> GND
- TP192 pad 1: /46 -> GND
- TP193 pad 1: /47 -> GND
- TP194 pad 1: /47 -> GND
- TP199 pad 1: /50 -> GND
- TP200 pad 1: /50 -> GND
- TP203 pad 1: /142 -> GND
- TP204 pad 1: /142 -> GND
- TP211 pad 1: /146 -> GND
- TP212 pad 1: /146 -> GND
- TP213 pad 1: /147 -> GND
- TP214 pad 1: /147 -> GND
- TP219 pad 1: /150 -> GND
- TP220 pad 1: /150 -> GND
- TP233 pad 1: /7 -> /43
- TP234 pad 1: /7 -> /43
- TP235 pad 1: /8 -> /31
- TP236 pad 1: /8 -> /31
- TP239 pad 1: /10 -> GND
- TP240 pad 1: /10 -> GND
- TP259 pad 1: /110 -> GND
- TP260 pad 1: /110 -> GND
- TP263 pad 1: /12 -> GND
- TP264 pad 1: /12 -> GND
- TP267 pad 1: /14 -> GND
- TP268 pad 1: /14 -> GND
- TP269 pad 1: /15 -> GND
- TP270 pad 1: /15 -> GND
- TP283 pad 1: /112 -> GND
- TP284 pad 1: /112 -> GND
- TP287 pad 1: /114 -> GND
- TP288 pad 1: /114 -> GND
- TP289 pad 1: /115 -> GND
- TP290 pad 1: /115 -> GND
Other:
- board text added: "GND"
- board text added: "Masse connecteurs (GND)"
- board text added: "Plan"
- board text added: "Plan de masse (Volant)"

Commit message: v0 near finished
Parts:
- added TPGND0: TestPoint, LibPersoNadj:Banana_test_point_4mm, F.Cu at (139.5, 172.0)
- added TPV0: TestPoint, LibPersoNadj:Banana_test_point_4mm, F.Cu at (120.5, 172.0)
- moved JMasse0 38.1 mm to (131.2, 148.5)
- moved SW1 10.0 mm to (90.0, 137.0)
- moved SW_Rej_A0 7.91 mm to (119.5, 72.5), turned to 270 degrees
- moved SW_RegB0 7.57 mm to (135.0, 72.5), turned to 270 degrees
- moved SW_Rej_C0 7.50 mm to (150.0, 72.5), turned to 270 degrees
- moved C1 6.50 mm to (29.5, 83.5)
- moved C2 6.26 mm to (29.5, 59.0)
- moved C3 6.26 mm to (29.5, 34.0)
- moved J12v0 5.10 mm to (135.0, 52.5)
- moved J_12v0 5.10 mm to (135.0, 42.5)
- moved J_Perturb1 5.00 mm to (150.0, 42.5)
- moved R1 5.00 mm to (155.0, 46.9)
- moved R10 5.00 mm to (145.9, 58.7)
- moved R11 5.00 mm to (149.3, 58.7)
- moved R12 5.00 mm to (144.9, 55.0)
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Other:
- board size 262.5 x 167.5 mm -> 267.5 x 170 mm
- board text added: "12V (Alim AOP)"
- board text added: "1=1A 50=50A"
- board text added: "Analyser 1"
- board text added: "Analyser 2"
- board text added: "Analyser 3"
- board text added: "Antenna"
- board text added: "DPU"
- board text added: "Disable|Enable (DC Removal)"
- board text added: "Enable|Disable"
- board text added: "Floating plane"
- board text added: "Ground (GND)"
- board text added: "Manual | Matrix"
- board text added: "Output"
- board text added: "Rejection cirtuit"
- board text added: "Ripple Input"
- board text added: "S | RTN"
- board text added: "Switch matrix"
- board text added: "Sy | RTNy"
- board text added: "Sz | RTNz"
- board text added: "Transfer fonction In"
- board text added: "Transfer fonction Out"
- board text added: "X|Y|Z"
- board text removed: "12V"
- board text removed: "Analyseur 1"
- board text removed: "Analyseur 2"
- board text removed: "Analyseur 3"
- board text removed: "Fonction transfer In"
- board text removed: "Fonction transfer Out"
- board text removed: "Manuel"
- board text removed: "Masse connecteurs (GND)"
- board text removed: "Matrice"
- board text removed: "Normal"
- board text removed: "Plan"
- board text removed: "Plan de masse (Volant)"
- board text removed: "Réjection"
- board text removed: "S X Y RTN Z"
- board text removed: "Sy RTNy"
- board text removed: "Sz RTNz"
- board text removed: "Test réjection"

Commit message: Pre-routage
Parts:
- added H5: MountingHole, MountingHole:MountingHole_3.2mm_M3, F.Cu at (137.5, 165.0)
- added H6: MountingHole, MountingHole:MountingHole_3.2mm_M3, F.Cu at (137.5, 5.00)
- moved H3 20.2 mm to (265.0, 5.00)
- moved H4 17.7 mm to (5.00, 5.00)
- moved H2 16.8 mm to (265.0, 165.0)
- moved JMasse0 16.8 mm to (138.8, 133.5)
- moved TPGND0 16.8 mm to (147.0, 157.0)
- moved TPV0 16.8 mm to (128.0, 157.0)
- moved J1 15.2 mm to (232.9, 120.5)
- moved J26 15.2 mm to (189.7, 120.5)
- moved R5 15.2 mm to (148.5, 31.8)
- moved R6 15.2 mm to (150.2, 31.8)
- moved C1 15.2 mm to (32.0, 68.5)
- moved C2 15.2 mm to (32.0, 44.0)
- moved C3 15.2 mm to (32.0, 19.0)
- moved J11 15.2 mm to (232.9, 92.6)
- moved J12v0 15.2 mm to (137.5, 37.5)
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Other:
- board size 267.5 x 170 mm -> 270 x 170 mm
- board text added: "12V"
- board text added: "Rejection circuit"
- board text added: "Transfer function Input"
- board text added: "Transfer function Output"
- board text removed: "12V (Alim AOP)"
- board text removed: "Rejection cirtuit"
- board text removed: "Transfer fonction In"
- board text removed: "Transfer fonction Out"
