File: CarteCaracTo/10PinSwichSides.sch (KiCad schematic (older format))
At the start: 0 parts

Commit message: Envoyé en prod
Changed lines of the file:
@@
 	2900 4150 3225 4150
 Wire Wire Line
-	2925 4900 3250 4900
+	2900 4900 3225 4900
 Wire Wire Line
 	2900 2300 3225 2300
@@
 Text HLabel 2900 4550 0    50   Input ~ 0
 8
-Text HLabel 2925 4900 0    50   Input ~ 0
+Text HLabel 2900 4900 0    50   Input ~ 0
 9
 Text HLabel 2900 5250 0    50   Input ~ 0
