File: CarteCarac/CaracAsic.sch (KiCad schematic (older format))
At the start: 2 parts

Commit message: Routé, verif pre-envoie
Changed lines of the file:
@@
 F15 "-R34" I R 2900 3875 50
 $EndSheet
-Text Label 9050 2325 2    50   ~ 0
+Text Label 8525 2325 0    50   ~ 0
 Pot_Offset_1
 Wire Wire Line
@@
 Wire Wire Line
 	9175 2725 8525 2725
-Text Label 9050 2425 2    50   ~ 0
+Text Label 8525 2425 0    50   ~ 0
 Pot_VDD_1
-Text Label 9050 2525 2    50   ~ 0
+Text Label 8525 2525 0    50   ~ 0
 Pot_Bias_1
-Text Label 9050 2725 2    50   ~ 0
+Text Label 8525 2725 0    50   ~ 0
 Pot_Offset_2
-Text Label 9050 2825 2    50   ~ 0
+Text Label 8525 2825 0    50   ~ 0
 Pot_VDD_2
-Text Label 9050 2925 2    50   ~ 0
+Text Label 8525 2925 0    50   ~ 0
 Pot_Bias_2
 Text Label 7100 1600 0    50   ~ 0

Commit message: Correction pinout 6P3T & ajout d'étiquettes sur pin hiérarchique 3P4T + routage
Changed lines of the file:
@@
-	-1   0    0    -1
-$EndComp
-$Comp
-L LibPersoNadj:SW_6P3T_Slide6x3 SW_Channels_0
-U 1 1 5E153517
-P 6575 2600
-AR Path="/5E153517" Ref="SW_Channels_0"  Part="1"
-AR Path="/5D6520CE/5E153517" Ref="SW_Channels_0"  Part="1"
-F 0 "SW_Channels_0" H 6625 3890 50  0000 C CNN
-F 1 "SW_6P3T_Slide6x3" H 6625 3799 50  0000 C CNN
-F 2 "LibPersoNadj:SW_6P3T_MSS6350R04_TE" H 6475 3900 50  0001 C CNN
-F 3 "http://cdn-reichelt.de/documents/datenblatt/C200/DS-Serie%23LOR.pdf" H 6475 3900 50  0001 C CNN
-	1    6575 2600
 	-1   0    0    -1
 $EndComp
@@
 AR Path="/5D9D35E7/5E076C40" Ref="#PWR?"  Part="1"
 F 0 "#PWR0142" H 7050 2350 50  0001 C CNN
-F 1 "GND" H 7055 2427 50  0000 C CNN
+F 1 "GND" V 7050 2375 50  0000 C CNN
 F 2 "" H 7050 2600 50  0001 C CNN
 F 3 "" H 7050 2600 50  0001 C CNN
@@
 Text HLabel 3600 4775 2    50   Input ~ 0
 -RZ10
+$Comp
+L LibPersoNadj:SW_6P3T_Slide6x3 SW_Channels_0
+U 1 1 5E7CD602
+P 6575 2600
+F 0 "SW_Channels_0" H 6625 3890 50  0000 C CNN
+F 1 "SW_6P3T_Slide6x3" H 6625 3799 50  0000 C CNN
+F 2 "LibPersoNadj:SW_6P3T_MSS6350R04_TE" H 6475 3900 50  0001 C CNN
+F 3 "http://cdn-reichelt.de/documents/datenblatt/C200/DS-Serie%23LOR.pdf" H 6475 3900 50  0001 C CNN
+	1    6575 2600
+	-1   0    0    -1
+$EndComp
 $EndSCHEMATC
