File: CarteCarac/CarteCarac.kicad_pcb (KiCad board)
At the start: 4 copper layers, 130 x 300 mm, 115 parts, among them J1 Conn_02x25_Top_Bottom_Mountin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, U1 ASIC_JUICE

Commit message: v0 near finished
Parts:
- removed CX1, CX2, CX3, CY1, CY2, CY3, CZ1, CZ2, CZ3: 680n, Capacitor_SMD:C_1812_4532Metric_Pad1.30x3.40mm_HandSolder
- removed CX10, CX12, CY10, CY12, CZ10, CZ12: 150p, Capacitor_SMD:C_0603_1608Metric_Pad1.05x0.95mm_HandSolder
- removed CX11, CX40, CY11, CY40, CZ11, CZ40: 220n, Capacitor_SMD:C_1206_3216Metric_Pad1.42x1.75mm_HandSolder
- removed CX13, CY13, CZ13: 220n/470n, Capacitor_SMD:C_1210_3225Metric_Pad1.42x2.65mm_HandSolder
- removed CX14, CY14, CZ14: 470n, Capacitor_SMD:C_1812_4532Metric_Pad1.30x3.40mm_HandSolder
- removed CX20, CX_CR1, CX_SC1, CX_SC2, CY20, CY_CR1, CY_SC1, CY_SC2, CZ20, CZ_CR1, CZ_SC1, CZ_SC2: TBD, Capacitor_SMD:C_0603_1608Metric_Pad1.05x0.95mm_HandSolder
- removed CX35, CX36, CX8, CY35, CY36, CY8, CZ35, CZ36, CZ8: 1n, Capacitor_SMD:C_0603_1608Metric_Pad1.05x0.95mm_HandSolder
- removed N_CFP64: Housing_Pad, TestPoint:TestPoint_Pad_4.0x4.0mm
- removed R1: 10k, Resistor_SMD:R_0603_1608Metric_Pad1.05x0.95mm_HandSolder
- removed RX10, RY10, RZ10: 22K, Resistor_SMD:R_0603_1608Metric_Pad1.05x0.95mm_HandSolder
- removed RX12, RY12, RZ12: 44K, Resistor_SMD:R_0603_1608Metric_Pad1.05x0.95mm_HandSolder
- removed RX14, RY14, RZ14: 100, Resistor_SMD:R_0603_1608Metric_Pad1.05x0.95mm_HandSolder
- removed RX20, RY20, RZ20: 68k, Resistor_SMD:R_0805_2012Metric_Pad1.15x1.40mm_HandSolder
- removed RX30, RY30, RZ30: 7,68k, Resistor_SMD:R_0603_1608Metric_Pad1.05x0.95mm_HandSolder
- removed RX31, RX33, RX41, RY31, RY33, RY41, RZ31, RZ33, RZ41: 49,9k, Resistor_SMD:R_0603_1608Metric_Pad1.05x0.95mm_HandSolder
- removed RX35, RX36, RY35, RY36, RZ35, RZ36: 49,9, Resistor_SMD:R_0603_1608Metric_Pad1.05x0.95mm_HandSolder
- removed RX40, RY40, RZ40: 750k, Resistor_SMD:R_1206_3216Metric_Pad1.42x1.75mm_HandSolder
- removed RX42, RY42, RZ42: 42,2k, Resistor_SMD:R_0603_1608Metric_Pad1.05x0.95mm_HandSolder
- removed RthB0: PT1000, Resistor_SMD:R_0603_1608Metric_Pad1.05x0.95mm_HandSolder
- removed U1: ASIC_JUICE, LibBurnInJuice:8500-50mm-64T-Ovale-EuroCircuitOK
- added H10: MountingHole_Pad, MountingHole:MountingHole_3.2mm_M3_Pad_Via, F.Cu at (-5.00, 60.0)
- added H9: MountingHole_Pad, MountingHole:MountingHole_3.2mm_M3_Pad_Via, F.Cu at (-5.00, -60.0)
- added J2: Conn_02x39_Top_Bottom_MountingPin, LibPersoNadj:db_78f_09565527613, F.Cu at (130.0, 0.00)
- moved H8 323.9 mm to (-110.0, -60.0), turned to 270 degrees
- moved J1 300.8 mm to (-122.0, 0.00), turned to 270 degrees
- moved RVX10 271.7 mm to (-75.0, -45.0), turned to 0 degrees
- moved H6 262.5 mm to (-110.0, 60.0), turned to 270 degrees
- moved RVY10 243.8 mm to (-75.0, -10.0), turned to 0 degrees
- moved SW_RX10 235.1 mm to (-40.0, -45.0), turned to 0 degrees
- moved RVZ10 223.6 mm to (-75.0, 25.0), turned to 0 degrees
- moved H7 217.1 mm to (130.0, -60.0), turned to 270 degrees
- moved RVX12 204.0 mm to (-5.00, -45.0), turned to 0 degrees
- moved SW_RY10 202.2 mm to (-40.0, -10.0), turned to 0 degrees
- moved SW_RX12 181.2 mm to (30.0, -45.0), turned to 0 degrees
- moved SW_Channels_0 179.5 mm to (-50.0, 53.0), turned to 0 degrees
- moved SW_RZ10 177.3 mm to (-40.0, 25.0), turned to 0 degrees
- moved SW_X32-34 173.3 mm to (100.0, -45.0), turned to 180 degrees
- moved RV_X32-34 170.3 mm to (65.0, -45.0), turned to 0 degrees
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Connections:
- J1 pad 16: Net-(J1-Pad16) -> /In2P_X
- J1 pad 17: /In2P_X -> /In2P_Y
- J1 pad 18: /In2P_Y -> /In2P_Z
- J1 pad 19: /In2P_Z -> /-RX10
- J1 pad 20: Net-(J1-Pad20) -> /-RY10
- J1 pad 21: Net-(J1-Pad21) -> /-RZ10
- J1 pad 22: Net-(J1-Pad22) -> /-RX12
- J1 pad 23: Net-(J1-Pad23) -> /-RY12
- J1 pad 24: Net-(J1-Pad24) -> /-RZ12
- SW_Channels_0 pad 1: /AsicFM/Pot_Offset_X_1 -> /CaracAsic/Pot_Offset_1
- SW_Channels_0 pad 10: /AsicFM/Pot_VDD_X_2 -> /CaracAsic/Pot_VDD_X_1
- SW_Channels_0 pad 11: /AsicFM/Pot_VDD_Y_2 -> /CaracAsic/Pot_VDD_Y_1
- SW_Channels_0 pad 12: /AsicFM/Pot_VDD_Z_2 -> /CaracAsic/Pot_VDD_Z_1
- SW_Channels_0 pad 13: /AsicFM/Pot_Bias_X_1 -> /CaracAsic/Pot_VDD_2
- SW_Channels_0 pad 14: /AsicFM/Pot_Bias_Y_1 -> /CaracAsic/Pot_VDD_X_2
- SW_Channels_0 pad 15: /AsicFM/Pot_Bias_Z_1 -> /CaracAsic/Pot_VDD_Y_2
- SW_Channels_0 pad 16: /AsicFM/Pot_Bias_X_2 -> /CaracAsic/Pot_VDD_Z_2
- SW_Channels_0 pad 17: /AsicFM/Pot_Bias_Y_2 -> /CaracAsic/Pot_Bias_1
- SW_Channels_0 pad 18: /AsicFM/Pot_Bias_Z_2 -> /CaracAsic/Pot_Bias_X_1
- SW_Channels_0 pad 19: /AsicFM/Pot_Offset_1 -> /CaracAsic/Pot_Bias_Y_1
- SW_Channels_0 pad 2: /AsicFM/Pot_Offset_Y_1 -> /CaracAsic/Pot_Offset_X_1
- SW_Channels_0 pad 20: /AsicFM/Pot_Offset_2 -> /CaracAsic/Pot_Bias_Z_1
- SW_Channels_0 pad 21: /AsicFM/Pot_VDD_1 -> /CaracAsic/Pot_Bias_2
- SW_Channels_0 pad 22: /AsicFM/Pot_VDD_2 -> /CaracAsic/Pot_Bias_X_2
- SW_Channels_0 pad 23: /AsicFM/Pot_Bias_1 -> /CaracAsic/Pot_Bias_Y_2
- SW_Channels_0 pad 24: /AsicFM/Pot_Bias_2 -> /CaracAsic/Pot_Bias_Z_2
- SW_Channels_0 pad 3: /AsicFM/Pot_Offset_Z_1 -> /CaracAsic/Pot_Offset_Y_1
- SW_Channels_0 pad 4: /AsicFM/Pot_Offset_X_2 -> /CaracAsic/Pot_Offset_Z_1
- SW_Channels_0 pad 5: /AsicFM/Pot_Offset_Y_2 -> /CaracAsic/Pot_Offset_2
- SW_Channels_0 pad 6: /AsicFM/Pot_Offset_Z_2 -> /CaracAsic/Pot_Offset_X_2
- SW_Channels_0 pad 7: /AsicFM/Pot_VDD_X_1 -> /CaracAsic/Pot_Offset_Y_2
- SW_Channels_0 pad 8: /AsicFM/Pot_VDD_Y_1 -> /CaracAsic/Pot_Offset_Z_2
- SW_Channels_0 pad 9: /AsicFM/Pot_VDD_Z_1 -> /CaracAsic/Pot_VDD_1
- SW_Pot_0 pad 1: /AsicFM/Pot_Offset_1 -> /CaracAsic/Pot_Offset_1
- SW_Pot_0 pad 3: /AsicFM/Pot_VDD_1 -> /CaracAsic/Pot_VDD_1
- SW_Pot_0 pad 4: /AsicFM/Pot_Bias_1 -> /CaracAsic/Pot_Bias_1
- SW_Pot_0 pad 5: /AsicFM/Pot_Offset_2 -> /CaracAsic/Pot_Offset_2
- SW_Pot_0 pad 7: /AsicFM/Pot_VDD_2 -> /CaracAsic/Pot_VDD_2
- SW_Pot_0 pad 8: /AsicFM/Pot_Bias_2 -> /CaracAsic/Pot_Bias_2
- SW_RX10 pad 1: /AsicFM/Pot_Bias_X_1 -> /CaracAsic/Pot_Bias_X_1
- SW_RX10 pad 3: Net-(RX10-Pad2) -> /+RX10
- SW_RX10 pad 4: /AsicFM/Pot_Bias_X_2 -> /CaracAsic/Pot_Bias_X_2
- SW_RX10 pad 6: /V_BIAS_LNA_X -> /-RX10
- SW_RX12 pad 1: /AsicFM/Pot_VDD_X_1 -> /CaracAsic/Pot_VDD_X_1
- SW_RX12 pad 3: Net-(RX12-Pad2) -> /+RX12
- SW_RX12 pad 4: /AsicFM/Pot_VDD_X_2 -> /CaracAsic/Pot_VDD_X_2
- SW_RX12 pad 6: /VDD_X -> /-RX12
- SW_RY10 pad 1: /AsicFM/Pot_Bias_Y_1 -> /CaracAsic/Pot_Bias_Y_1
- SW_RY10 pad 3: Net-(RY10-Pad2) -> /+RY10
- SW_RY10 pad 4: /AsicFM/Pot_Bias_Y_2 -> /CaracAsic/Pot_Bias_Y_2
- SW_RY10 pad 6: /V_BIAS_LNA_Y -> /-RY10
- SW_RY12 pad 1: /AsicFM/Pot_VDD_Y_1 -> /CaracAsic/Pot_VDD_Y_1
- SW_RY12 pad 3: Net-(RY12-Pad2) -> /+RY12
- SW_RY12 pad 4: /AsicFM/Pot_VDD_Y_2 -> /CaracAsic/Pot_VDD_Y_2
- SW_RY12 pad 6: /VDD_Y -> /-RY12
- SW_RZ10 pad 1: /AsicFM/Pot_Bias_Z_1 -> /CaracAsic/Pot_Bias_Z_1
- SW_RZ10 pad 3: Net-(RZ10-Pad2) -> /+RZ10
- SW_RZ10 pad 4: /AsicFM/Pot_Bias_Z_2 -> /CaracAsic/Pot_Bias_Z_2
- SW_RZ10 pad 6: /V_BIAS_LNA_Z -> /-RZ10
- SW_RZ12 pad 1: /AsicFM/Pot_VDD_Z_1 -> /CaracAsic/Pot_VDD_Z_1
- SW_RZ12 pad 3: Net-(RZ12-Pad2) -> /+RZ12
- SW_RZ12 pad 4: /AsicFM/Pot_VDD_Z_2 -> /CaracAsic/Pot_VDD_Z_2
- SW_RZ12 pad 6: /VDD_Z -> /-RZ12
- SW_X32-34 pad 1: /AsicFM/ChannelX/+32 -> /+RX32
- SW_X32-34 pad 10: /AsicFM/ChannelX/-34 -> /-RX34
- SW_X32-34 pad 11: /AsicFM/ChannelX/-34 -> /CaracAsic/ChannelX/-34
- SW_X32-34 pad 12: /AsicFM/In2N_X -> /CaracAsic/ChannelX/-32
- SW_X32-34 pad 15: /AsicFM/In2N_X -> /CaracAsic/ChannelX/In2N
- SW_X32-34 pad 16: /AsicFM/In2N_X -> /CaracAsic/ChannelX/In2N
- SW_X32-34 pad 2: /AsicFM/Pot_Offset_X_1 -> /CaracAsic/Pot_Offset_X_1
- SW_X32-34 pad 3: /AsicFM/In2N_X -> /CaracAsic/ChannelX/+34
- SW_X32-34 pad 4: /AsicFM/In2N_X -> /+RX34
- SW_X32-34 pad 5: /AsicFM/Pot_Offset_X_2 -> /CaracAsic/Pot_Offset_X_2
- SW_X32-34 pad 6: /AsicFM/ChannelX/-34 -> /CaracAsic/ChannelX/-34
- SW_X32-34 pad 7: /AsicFM/In2N_X -> /+RX34
- SW_X32-34 pad 8: /AsicFM/ChannelX/+32 -> /CaracAsic/ChannelX/+32
- SW_X32-34 pad 9: /AsicFM/ChannelX/+32 -> /CaracAsic/ChannelX/+32
- SW_Y32-34 pad 1: /AsicFM/ChannelY/+32 -> /+RY32
- SW_Y32-34 pad 10: /AsicFM/ChannelY/-34 -> /-RY34
- SW_Y32-34 pad 11: /AsicFM/ChannelY/-34 -> /CaracAsic/ChannelY/-34
- SW_Y32-34 pad 12: /AsicFM/In2N_Y -> /CaracAsic/ChannelY/-32
- SW_Y32-34 pad 15: /AsicFM/In2N_Y -> /CaracAsic/ChannelY/In2N
- SW_Y32-34 pad 16: /AsicFM/In2N_Y -> /CaracAsic/ChannelY/In2N
- SW_Y32-34 pad 2: /AsicFM/Pot_Offset_Y_1 -> /CaracAsic/Pot_Offset_Y_1
- SW_Y32-34 pad 3: /AsicFM/In2N_Y -> /CaracAsic/ChannelY/+34
- SW_Y32-34 pad 4: /AsicFM/In2N_Y -> /+RY34
- SW_Y32-34 pad 5: /AsicFM/Pot_Offset_Y_2 -> /CaracAsic/Pot_Offset_Y_2
- SW_Y32-34 pad 6: /AsicFM/ChannelY/-34 -> /CaracAsic/ChannelY/-34
- SW_Y32-34 pad 7: /AsicFM/In2N_Y -> /+RY34
- SW_Y32-34 pad 8: /AsicFM/ChannelY/+32 -> /CaracAsic/ChannelY/+32
- SW_Y32-34 pad 9: /AsicFM/ChannelY/+32 -> /CaracAsic/ChannelY/+32
- SW_Z32-34 pad 1: /AsicFM/ChannelZ/+32 -> /+RZ32
- SW_Z32-34 pad 10: /AsicFM/ChannelZ/-34 -> /-RZ34
- SW_Z32-34 pad 11: /AsicFM/ChannelZ/-34 -> /CaracAsic/ChannelZ/-34
- SW_Z32-34 pad 12: /AsicFM/In2N_Z -> /CaracAsic/ChannelZ/-32
- SW_Z32-34 pad 15: /AsicFM/In2N_Z -> /CaracAsic/ChannelZ/In2N
- SW_Z32-34 pad 16: /AsicFM/In2N_Z -> /CaracAsic/ChannelZ/In2N
- SW_Z32-34 pad 2: /AsicFM/Pot_Offset_Z_1 -> /CaracAsic/Pot_Offset_Z_1
- SW_Z32-34 pad 3: /AsicFM/In2N_Z -> /CaracAsic/ChannelZ/+34
- SW_Z32-34 pad 4: /AsicFM/In2N_Z -> /+RZ34
- SW_Z32-34 pad 5: /AsicFM/Pot_Offset_Z_2 -> /CaracAsic/Pot_Offset_Z_2
- SW_Z32-34 pad 6: /AsicFM/ChannelZ/-34 -> /CaracAsic/ChannelZ/-34
- SW_Z32-34 pad 7: /AsicFM/In2N_Z -> /+RZ34
- SW_Z32-34 pad 8: /AsicFM/ChannelZ/+32 -> /CaracAsic/ChannelZ/+32
- SW_Z32-34 pad 9: /AsicFM/ChannelZ/+32 -> /CaracAsic/ChannelZ/+32
Routing:
- net /+6V_C: track 76.5 -> 0.00 mm
- net /+6V_B: track 75.0 -> 0.00 mm, vias 2 -> 0
- net /VDD_Y: track 71.2 -> 0.00 mm
- net /V_BIAS_LNA_Y: track 64.5 -> 0.00 mm, vias 1 -> 0
- net /M_Y: track 62.6 -> 0.00 mm, vias 1 -> 0
- net /VDD_Z: track 57.9 -> 0.00 mm, vias 1 -> 0
- net /V_BIAS_LNA_Z: track 54.9 -> 0.00 mm, vias 1 -> 0
- net /Sy: track 54.5 -> 0.00 mm, vias 1 -> 0
- net /CR_Y: track 54.0 -> 0.00 mm, vias 2 -> 0
- net /AsicFM/Regu_Bias_LNA_Y: track 53.6 -> 0.00 mm, vias 2 -> 0
- net /CR_Z: track 53.3 -> 0.00 mm, vias 1 -> 0
- net /AsicFM/ChannelY/+32: track 46.0 -> 0.00 mm, vias 1 -> 0
- net /AsicFM/CAL_In_Z: track 44.9 -> 0.00 mm, vias 1 -> 0
- net /AsicFM/Regu_VDD_Y: track 44.6 -> 0.00 mm, vias 2 -> 0
- net /M_Z: track 43.8 -> 0.00 mm
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Other:
- board size 130 x 300 mm -> 250 x 130 mm
- board text added: "Mesure ---- Reglage"
- board text added: "Offset X"
- board text added: "Offset Y"
- board text added: "Offset Z"
- board text added: "Rise|c-c|Drop measure"
- board text added: "VDD X"
- board text added: "VDD Y"
- board text added: "VDD Z"
- board text added: "V_Bias X"
- board text added: "V_Bias Y"
- board text added: "V_Bias Z"
- board text added: "V_Bias | VDD | Offset"
- board text added: "X|Y|Z"

Commit message: Pre-routage
Parts:
- moved SW_RX12 3.16 mm to (31.0, -48.0)
- moved SW_RY12 2.24 mm to (31.0, -12.0)
- moved SW_RZ12 2.24 mm to (31.0, 23.0)
- moved SW_Z32-34 2.00 mm to (100.0, 25.0)
Other:
- board text added: "Pins: 64 & 65 Pins: 66 & 64"
- board text added: "Pins: 67 & 22"
- board text added: "Pins: 68 & 19"
- board text added: "Pins: 69 & 70 Pins: 71 & 69"
- board text added: "Pins: 72 & 23"
- board text added: "Pins: 73 & 20"
- board text added: "Pins: 74 & 75 Pins: 76 & 74"
- board text added: "Pins: 77 & 24"
- board text added: "Pins: 78 & 21"

Commit message: cleaning Pre-routage
Parts:
- moved SW_RX10 2.24 mm to (-39.0, -47.0)
- moved SW_RY10 2.24 mm to (-39.0, -12.0)
- moved SW_RZ10 2.24 mm to (-39.0, 23.0)
- moved SW_X32-34 1.00 mm to (100.0, -46.0)
- moved SW_Y32-34 1.00 mm to (100.0, -11.0)
- moved SW_Z32-34 1.00 mm to (100.0, 24.0)
Changed lines of the file:
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@@
   )
   (module LibPersoNadj:Switch_4P3T_MRA403_NKK_Turned30° (layer F.Cu)
-    (at 100 25 180)
+    (at 100 24 180)
     (descr "4P3T MRA403 NKK")
     (tags "Switch 4P3T MRA403 NKK")
@@
   )
   (module LibPersoNadj:Switch_4P3T_MRA403_NKK_Turned30° (layer F.Cu)
-    (at 100 -10 180)
+    (at 100 -11 180)
     (descr "4P3T MRA403 NKK")
     (tags "Switch 4P3T MRA403 NKK")
@@
   )
   (module LibPersoNadj:Switch_4P3T_MRA403_NKK_Turned30° (layer F.Cu)
-    (at 100 -45 180)
+    (at 100 -46 180)
     (descr "4P3T MRA403 NKK")
     (tags "Switch 4P3T MRA403 NKK")
@@
   )
   (module LibPersoNadj:SW_NKK_DPDT_B22AP (layer F.Cu)
-    (at -40 25)
+    (at -39 23)
     (descr "Switch NKK DPDT http://www.nkkswitches.com/pdf/Btoggles.pdf")
     (tags "SWITCH TOGGLE DPDT")
@@
   )
   (module LibPersoNadj:SW_NKK_DPDT_B22AP (layer F.Cu)
-    (at -40 -10)
+    (at -39 -12)
     (descr "Switch NKK DPDT http://www.nkkswitches.com/pdf/Btoggles.pdf")
     (tags "SWITCH TOGGLE DPDT")
@@
   )
   (module LibPersoNadj:SW_NKK_DPDT_B22AP (layer F.Cu)
-    (at -40 -45)
+    (at -39 -47)
     (descr "Switch NKK DPDT http://www.nkkswitches.com/pdf/Btoggles.pdf")
     (tags "SWITCH TOGGLE DPDT")
@@
   (gr_line (start 85 10) (end 85 5.5) (layer F.SilkS) (width 0.12))
   (gr_line (start 85 5.5) (end 105 5.5) (layer F.SilkS) (width 0.12))
-  (gr_line (start 105 -29.5) (end 105 -25) (layer F.SilkS) (width 0.12))
-  (gr_line (start 85 -29.5) (end 105 -29.5) (layer F.SilkS) (width 0.12))
+  (gr_line (start 105 -30.5) (end 105 -26) (layer F.SilkS) (width 0.12))
+  (gr_line (start 85 -30.5) (end 105 -30.5) (layer F.SilkS) (width 0.12))
   (gr_line (start 85 -25) (end 85 -29.5) (layer F.SilkS) (width 0.12))
   (gr_line (start 37.5 -4) (end 14.5 -4) (layer F.SilkS) (width 0.12))
@@
   (gr_line (start -95 -32.5) (end -32.5 -32.5) (layer F.SilkS) (width 0.12))
   (gr_line (start -95 -57.5) (end -95 -32.5) (layer F.SilkS) (width 0.12))
-  (gr_line (start 96.3 -36) (end 97.2 -36.9) (layer F.SilkS) (width 0.3))
-  (gr_text " Rise|c-c|Drop\n measure\n" (at 99.7 -33) (layer F.SilkS)
+  (gr_line (start 96.3 -37) (end 97.2 -37.9) (layer F.SilkS) (width 0.3))
+  (gr_text " Rise|c-c|Drop\n measure\n" (at 99.7 -34) (layer F.SilkS)
     (effects (font (size 2 2) (thickness 0.3)))
   )
-  (gr_line (start 104.1 -36) (end 103.1 -37) (layer F.SilkS) (width 0.3))
-  (gr_arc (start 96.289378 -29.082184) (end 96.289378 -33.082184) (angle -50) (layer F.SilkS) (width 0.3))
-  (gr_arc (start 104.100622 -29.082184) (end 104.100622 -33.082184) (angle 50) (layer F.SilkS) (width 0.3))
-  (gr_line (start 96.3 -1) (end 97.2 -1.9) (layer F.SilkS) (width 0.3))
-  (gr_text " Rise|c-c|Drop\n measure\n" (at 99.7 2) (layer F.SilkS)
+  (gr_line (start 104.1 -37) (end 103.1 -38) (layer F.SilkS) (width 0.3))
+  (gr_arc (start 96.289378 -30.082184) (end 96.289378 -34.082184) (angle -50) (layer F.SilkS) (width 0.3))
+  (gr_arc (start 104.100622 -30.082184) (end 104.100622 -34.082184) (angle 50) (layer F.SilkS) (width 0.3))
+  (gr_line (start 96.3 -2) (end 97.2 -2.9) (layer F.SilkS) (width 0.3))
+  (gr_text " Rise|c-c|Drop\n measure\n" (at 99.7 1) (layer F.SilkS)
     (effects (font (size 2 2) (thickness 0.3)))
   )
-  (gr_line (start 104.1 -1) (end 103.1 -2) (layer F.SilkS) (width 0.3))
-  (gr_arc (start 96.289378 5.917816) (end 96.289378 1.917816) (angle -50) (layer F.SilkS) (width 0.3))
-  (gr_arc (start 104.100622 5.917816) (end 104.100622 1.917816) (angle 50) (layer F.SilkS) (width 0.3))
-  (gr_line (start 96.3 34) (end 97.2 33.1) (layer F.SilkS) (width 0.3))
-  (gr_line (start 104.1 34) (end 103.1 33) (layer F.SilkS) (width 0.3))
-  (gr_arc (start 96.289378 40.917816) (end 96.289378 36.917816) (angle -50) (layer F.SilkS) (width 0.3))
-  (gr_arc (start 104.100622 40.917816) (end 104.100622 36.917816) (angle 50) (layer F.SilkS) (width 0.3))
-  (gr_text " Rise|c-c|Drop\n measure\n" (at 99.7 37) (layer F.SilkS)
+  (gr_line (start 104.1 -2) (end 103.1 -3) (layer F.SilkS) (width 0.3))
+  (gr_arc (start 96.289378 4.917816) (end 96.289378 0.917816) (angle -50) (layer F.SilkS) (width 0.3))
+  (gr_arc (start 104.100622 4.917816) (end 104.100622 0.917816) (angle 50) (layer F.SilkS) (width 0.3))
+  (gr_line (start 96.3 33) (end 97.2 32.1) (layer F.SilkS) (width 0.3))
+  (gr_line (start 104.1 33) (end 103.1 32) (layer F.SilkS) (width 0.3))
+  (gr_arc (start 96.289378 39.917816) (end 96.289378 35.917816) (angle -50) (layer F.SilkS) (width 0.3))
+  (gr_arc (start 104.100622 39.917816) (end 104.100622 35.917816) (angle 50) (layer F.SilkS) (width 0.3))
+  (gr_text " Rise|c-c|Drop\n measure\n" (at 99.7 36) (layer F.SilkS)
     (effects (font (size 2 2) (thickness 0.3)))
   )
@@
     (effects (font (size 2 2) (thickness 0.3)))
   )
-  (gr_text "Mesure\n----\nReglage" (at -50.5 -45) (layer F.SilkS)
+  (gr_text "Mesure\n----\nReglage" (at -49.5 -47) (layer F.SilkS)
     (effects (font (size 2 2) (thickness 0.3)))
   )
-  (gr_text "Mesure\n----\nReglage" (at -50.5 -10) (layer F.SilkS)
+  (gr_text "Mesure\n----\nReglage" (at -49.5 -12) (layer F.SilkS)
     (effects (font (size 2 2) (thickness 0.3)))
   )
@@
     (effects (font (size 3 3) (thickness 0.45)))
   )
-  (gr_text "Mesure\n----\nReglage" (at -50.5 25) (layer F.SilkS)
+  (gr_text "Mesure\n----\nReglage" (at -49.5 23) (layer F.SilkS)
     (effects (font (size 2 2) (thickness 0.3)))
   )

Commit message: Routé, verif pre-envoie
Parts:
- J_50m_1: renamed from J1; footprint LibPersoNadj:DD50S564TLF -> LibPersoNadj:db_50m_MP_DD50S564TXLF
- J_78f_1: renamed from J2; footprint LibPersoNadj:db_78f_09565527613 -> LibPersoNadj:db_78f_MP_09565527613
Connections:
- net /RTNx renamed Sx-
- net /RTNy renamed Sy-
- net /RTNz renamed Sz-
- net /Sx renamed Sx+
- net /Sy renamed Sy+
- J_50m_1 pad 29: /Sz -> Sz+
- J_50m_1 pad 9: /M_X -> Sz+
- J_78f_1 pad 10: GND -> Sz+
- J_78f_1 pad 29: /Sz -> Sz+
- J_78f_1 pad 9: /M_X -> Sz+
- SW_X32-34 pad 11: /CaracAsic/ChannelX/-34 -> /-RX34
- SW_X32-34 pad 12: /CaracAsic/ChannelX/-32 -> /+RX34
- SW_X32-34 pad 15: /CaracAsic/ChannelX/In2N -> /+RX34
- SW_X32-34 pad 16: /CaracAsic/ChannelX/In2N -> /+RX34
- SW_X32-34 pad 3: /CaracAsic/ChannelX/+34 -> /+RX34
- SW_X32-34 pad 6: /CaracAsic/ChannelX/-34 -> /-RX34
- SW_Y32-34 pad 11: /CaracAsic/ChannelY/-34 -> /-RY34
- SW_Y32-34 pad 12: /CaracAsic/ChannelY/-32 -> /+RY34
- SW_Y32-34 pad 15: /CaracAsic/ChannelY/In2N -> /+RY34
- SW_Y32-34 pad 16: /CaracAsic/ChannelY/In2N -> /+RY34
- SW_Y32-34 pad 3: /CaracAsic/ChannelY/+34 -> /+RY34
- SW_Y32-34 pad 6: /CaracAsic/ChannelY/-34 -> /-RY34
- SW_Z32-34 pad 11: /CaracAsic/ChannelZ/-34 -> /-RZ34
- SW_Z32-34 pad 12: /CaracAsic/ChannelZ/-32 -> /+RZ34
- SW_Z32-34 pad 15: /CaracAsic/ChannelZ/In2N -> /+RZ34
- SW_Z32-34 pad 16: /CaracAsic/ChannelZ/In2N -> /+RZ34
- SW_Z32-34 pad 3: /CaracAsic/ChannelZ/+34 -> /+RZ34
- SW_Z32-34 pad 6: /CaracAsic/ChannelZ/-34 -> /-RZ34
Routing:
- net Sz+: track 0.00 -> 451.2 mm
- net /Temp_Mon_B: track 0.00 -> 336.5 mm
- net /+6V_C: track 0.00 -> 302.2 mm
- net /-RZ10: track 0.00 -> 295.6 mm, vias 0 -> 2
- net /+6V_A: track 0.00 -> 285.9 mm, vias 0 -> 3
- net /-RX12: track 0.00 -> 281.7 mm, vias 0 -> 3
- net /-RX10: track 0.00 -> 278.7 mm, vias 0 -> 2
- net /CAL: track 0.00 -> 272.4 mm
- net Sy-: track 0.00 -> 270.3 mm
- net /Temp_Mon_A: track 0.00 -> 265.2 mm, vias 0 -> 1
- net /RTN_Mon_A: track 0.00 -> 263.9 mm, vias 0 -> 1
- net /-RZ12: track 0.00 -> 261.5 mm, vias 0 -> 2
- net Sy+: track 0.00 -> 259.5 mm
- net /+6V_B: track 0.00 -> 254.7 mm, vias 0 -> 2
- net /-RY10: track 0.00 -> 254.6 mm, vias 0 -> 3
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- added copper zone on B.Cu, net GND
- added copper zone on F.Cu, net GND
- added copper zone on In1.Cu, net GND
- added copper zone on In2.Cu, net GND
Other:
- net class Default: clearance 0.15 -> 0.2; trace_width 0.2 -> 0.25
- rule trace_clearance: 0.15 -> 0.2
- rule trace_min: 0.15 -> 0.25

Commit message: Envoyé en prod
Connections:
- J_50m_1 pad 9: Sz+ -> /M_X
- J_78f_1 pad 10: Sz+ -> GND
- J_78f_1 pad 9: Sz+ -> /M_X
Routing:
- net Sz+: track 451.2 -> 230.3 mm
- net /M_X: track 0.00 -> 220.8 mm

Commit message: Correction pinout 6P3T & ajout d'étiquettes sur pin hiérarchique 3P4T + routage
Parts:
- RVX10, RVY10, RVZ10: value 12K -> 20K
- RVX12, RVY12, RVZ12: value 16K -> 20K
Connections:
- SW_Channels_0 pad 1: /CaracAsic/Pot_Offset_1 -> /CaracAsic/Pot_Offset_X_1
- SW_Channels_0 pad 10: /CaracAsic/Pot_VDD_X_1 -> /CaracAsic/Pot_VDD_1
- SW_Channels_0 pad 13: /CaracAsic/Pot_VDD_2 -> /CaracAsic/Pot_VDD_X_2
- SW_Channels_0 pad 14: /CaracAsic/Pot_VDD_X_2 -> /CaracAsic/Pot_VDD_2
- SW_Channels_0 pad 17: /CaracAsic/Pot_Bias_1 -> /CaracAsic/Pot_Bias_X_1
- SW_Channels_0 pad 18: /CaracAsic/Pot_Bias_X_1 -> /CaracAsic/Pot_Bias_1
- SW_Channels_0 pad 2: /CaracAsic/Pot_Offset_X_1 -> /CaracAsic/Pot_Offset_1
- SW_Channels_0 pad 21: /CaracAsic/Pot_Bias_2 -> /CaracAsic/Pot_Bias_X_2
- SW_Channels_0 pad 22: /CaracAsic/Pot_Bias_X_2 -> /CaracAsic/Pot_Bias_2
- SW_Channels_0 pad 5: /CaracAsic/Pot_Offset_2 -> /CaracAsic/Pot_Offset_X_2
- SW_Channels_0 pad 6: /CaracAsic/Pot_Offset_X_2 -> /CaracAsic/Pot_Offset_2
- SW_Channels_0 pad 9: /CaracAsic/Pot_VDD_1 -> /CaracAsic/Pot_VDD_X_1
- SW_X32-34 pad 8: /CaracAsic/ChannelX/+32 -> /+RX32
- SW_X32-34 pad 9: /CaracAsic/ChannelX/+32 -> /+RX32
- SW_Y32-34 pad 8: /CaracAsic/ChannelY/+32 -> /+RY32
- SW_Y32-34 pad 9: /CaracAsic/ChannelY/+32 -> /+RY32
- SW_Z32-34 pad 8: /CaracAsic/ChannelZ/+32 -> /+RZ32
- SW_Z32-34 pad 9: /CaracAsic/ChannelZ/+32 -> /+RZ32
Routing:
- net /CaracAsic/Pot_Bias_X_2: track 144.4 -> 128.8 mm
- net /CaracAsic/Pot_Bias_1: track 100.7 -> 87.4 mm, vias 1 -> 0
- net /+RZ32: track 41.2 -> 52.7 mm
- net /+RX32: track 70.4 -> 81.8 mm
- net /+RY32: track 78.8 -> 90.3 mm
- net /CaracAsic/Pot_Bias_Z_1: track 38.6 -> 46.2 mm
- net /CaracAsic/Pot_VDD_X_1: track 131.9 -> 138.7 mm, vias 0 -> 1
- net /-RZ10: track 295.6 -> 291.3 mm
- net /CaracAsic/Pot_VDD_X_2: track 199.1 -> 203.1 mm
- net /CaracAsic/Pot_Bias_2: track 81.1 -> 77.8 mm
- net /CaracAsic/Pot_Offset_2: track 107.6 -> 104.6 mm
- net /CaracAsic/Pot_VDD_2: track 105.5 -> 102.6 mm
- net /CaracAsic/ChannelX/+32: track 2.64 -> 0.00 mm
- net /CaracAsic/ChannelZ/+32: track 2.64 -> 0.00 mm
- net /CaracAsic/ChannelY/+32: track 2.64 -> 0.00 mm
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